File: ADC.kicad_sch (KiCad schematic)
At the start: 22 parts, among them J22 AIN, U17 ADS1115IDGS

Commit message: layout
Parts:
- removed D10, D12, D8: D_Zener, Diode_SMD:D_SMA-SMB_Universal_Handsoldering, symbol Device:D_Zener
- removed D11, D5, D6, D7, D9: D_Schottky, Diode_SMD:D_SMA-SMB_Universal_Handsoldering, symbol Device:D_Schottky
- removed JP10: A2, Jumper:SolderJumper-2_P1.3mm_Open_Pad1.0x1.5mm, symbol Jumper:SolderJumper_2_Open
- removed JP11: A3, Jumper:SolderJumper-2_P1.3mm_Open_Pad1.0x1.5mm, symbol Jumper:SolderJumper_2_Open
- removed JP9: A1, Jumper:SolderJumper-2_P1.3mm_Open_Pad1.0x1.5mm, symbol Jumper:SolderJumper_2_Open
- added D2102, D2103, D2104, D2105, D2106, D2107, D2108, D2109: 1N5819, Diode_SMD:D_SOD-323, symbol Diode:1N5819
- R1201: renamed from R66; value R -> 12k
- R1202: renamed from R67; value R -> 1k5
- R1203: renamed from R68; value R -> 12k
- R1204: renamed from R69; value R -> 1k5
- R1205: renamed from R70; value R -> 12k
- R1206: renamed from R71; value R -> 1k5
- R1207: renamed from R72; value R -> 12k
- R1208: renamed from R73; value R -> 1k5
- renumbered C44 to C1201, J22 to J1201, U17 to U1201
Connections:
- net +3V3: now also D2102.1 (K), D2104.1 (K), D2106.1 (K), D2108.1 (K)
- net GND: now also D2103.2 (A), D2105.2 (A), D2107.2 (A), D2109.2 (A)
- net at R1201.2, R1202.1, U1201.4 (AIN0): now also D2102.2 (A), D2103.1 (K)
- net at R1203.2, R1204.1, U1201.5 (AIN1): now also D2104.2 (A), D2105.1 (K)
- net at R1205.2, R1206.1, U1201.6 (AIN2): now also D2106.2 (A), D2107.1 (K)
- net at R1207.2, R1208.1, U1201.7 (AIN3): now also D2108.2 (A), D2109.1 (K)
Other:
- note added: "AIN=(UIN*RGND)/(RIN+RGND) (28*1500)/(12000+1500)=3.2V"
