File: AMP.kicad_sch (KiCad schematic)
At the start: 11 parts, among them U14 LM324

Commit message: layout
Parts:
- JP701: renamed from JP8; value Jumper_3_Open -> DAC AMP
- R701: renamed from R25; value R -> 10k
- R702: renamed from R26; value R -> 10k
- R703: renamed from R27; value R -> 68k
- R704: renamed from R28; value R -> 68k
- R705: renamed from R29; value R -> 10k
- R706: renamed from R30; value R -> 10k
- R707: renamed from R31; value R -> 68k
- R708: renamed from R32; value R -> 68k
- renumbered C28 to C701, U14 to U701
Changed lines of the file:
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@@
   (symbol (lib_id "Device:R") (at 171.45 73.66 90) (unit 1)
     (in_bom yes) (on_board yes)
-    (property "Reference" "R26" (id 0) (at 171.45 78.9178 90))
-    (property "Value" "R" (id 1) (at 171.45 76.6064 90))
+    (property "Reference" "R702" (id 0) (at 171.45 78.9178 90))
+    (property "Value" "10k" (id 1) (at 171.45 76.6064 90))
     (property "Footprint" "Resistor_SMD:R_0603_1608Metric" (id 2) (at 171.45 75.438 90)
       (effects (font (size 1.27 1.27)) hide)
@@
   (symbol (lib_id "Device:C") (at 165.1 177.8 0) (unit 1)
     (in_bom yes) (on_board yes)
-    (property "Reference" "C28" (id 0) (at 168.021 176.6316 0)
+    (property "Reference" "C701" (id 0) (at 168.021 176.6316 0)
       (effects (font (size 1.27 1.27)) (justify left))
     )
@@
   (symbol (lib_id "Device:R") (at 187.96 78.74 90) (unit 1)
     (in_bom yes) (on_board yes)
-    (property "Reference" "R28" (id 0) (at 187.96 83.9978 90))
-    (property "Value" "R" (id 1) (at 187.96 81.6864 90))
+    (property "Reference" "R704" (id 0) (at 187.96 83.9978 90))
+    (property "Value" "68k" (id 1) (at 187.96 81.6864 90))
     (property "Footprint" "Resistor_SMD:R_0603_1608Metric" (id 2) (at 187.96 80.518 90)
       (effects (font (size 1.27 1.27)) hide)
@@
   (symbol (lib_id "Amplifier_Operational:LM324") (at 114.3 71.12 0) (unit 1)
     (in_bom yes) (on_board yes)
-    (property "Reference" "U14" (id 0) (at 114.3 61.7982 0))
+    (property "Reference" "U701" (id 0) (at 114.3 61.7982 0))
     (property "Value" "LM324" (id 1) (at 114.3 64.1096 0))
     (property "Footprint" "Package_SO:SOIC-14_3.9x8.7mm_P1.27mm" (id 2) (at 113.03 68.58 0)
@@
   (symbol (lib_id "Amplifier_Operational:LM324") (at 187.96 71.12 0) (unit 2)
     (in_bom yes) (on_board yes)
-    (property "Reference" "U14" (id 0) (at 187.96 61.7982 0))
+    (property "Reference" "U701" (id 0) (at 187.96 61.7982 0))
     (property "Value" "LM324" (id 1) (at 187.96 64.1096 0))
     (property "Footprint" "Package_SO:SOIC-14_3.9x8.7mm_P1.27mm" (id 2) (at 186.69 68.58 0)
@@
   (symbol (lib_id "Amplifier_Operational:LM324") (at 114.3 114.3 0) (unit 3)
     (in_bom yes) (on_board yes)
-    (property "Reference" "U14" (id 0) (at 114.3 104.9782 0))
+    (property "Reference" "U701" (id 0) (at 114.3 104.9782 0))
     (property "Value" "LM324" (id 1) (at 114.3 107.2896 0))
     (property "Footprint" "Package_SO:SOIC-14_3.9x8.7mm_P1.27mm" (id 2) (at 113.03 111.76 0)
@@
   (symbol (lib_id "Amplifier_Operational:LM324") (at 187.96 114.3 0) (unit 4)
     (in_bom yes) (on_board yes)
-    (property "Reference" "U14" (id 0) (at 187.96 104.9782 0))
+    (property "Reference" "U701" (id 0) (at 187.96 104.9782 0))
     (property "Value" "LM324" (id 1) (at 187.96 107.2896 0))
     (property "Footprint" "Package_SO:SOIC-14_3.9x8.7mm_P1.27mm" (id 2) (at 186.69 111.76 0)
@@
   (symbol (lib_id "Amplifier_Operational:LM324") (at 153.67 177.8 0) (unit 5)
     (in_bom yes) (on_board yes)
-    (property "Reference" "U14" (id 0) (at 152.6032 176.6316 0)
+    (property "Reference" "U701" (id 0) (at 152.6032 176.6316 0)
       (effects (font (size 1.27 1.27)) (justify left))
     )
@@
   (symbol (lib_id "Device:R") (at 114.3 78.74 90) (unit 1)
     (in_bom yes) (on_board yes)
-    (property "Reference" "R27" (id 0) (at 114.3 83.9978 90))
-    (property "Value" "R" (id 1) (at 114.3 81.6864 90))
+    (property "Reference" "R703" (id 0) (at 114.3 83.9978 90))
+    (property "Value" "68k" (id 1) (at 114.3 81.6864 90))
     (property "Footprint" "Resistor_SMD:R_0603_1608Metric" (id 2) (at 114.3 80.518 90)
       (effects (font (size 1.27 1.27)) hide)
@@
   (symbol (lib_id "Device:R") (at 97.79 73.66 90) (unit 1)
     (in_bom yes) (on_board yes)
-    (property "Reference" "R25" (id 0) (at 97.79 78.9178 90))
-    (property "Value" "R" (id 1) (at 97.79 76.6064 90))
+    (property "Reference" "R701" (id 0) (at 97.79 78.9178 90))
+    (property "Value" "10k" (id 1) (at 97.79 76.6064 90))
     (property "Footprint" "Resistor_SMD:R_0603_1608Metric" (id 2) (at 97.79 75.438 90)
       (effects (font (size 1.27 1.27)) hide)
@@
   (symbol (lib_id "Device:R") (at 114.3 121.92 90) (unit 1)
     (in_bom yes) (on_board yes)
-    (property "Reference" "R31" (id 0) (at 114.3 127.1778 90))
-    (property "Value" "R" (id 1) (at 114.3 124.8664 90))
+    (property "Reference" "R707" (id 0) (at 114.3 127.1778 90))
+    (property "Value" "68k" (id 1) (at 114.3 124.8664 90))
     (property "Footprint" "Resistor_SMD:R_0603_1608Metric" (id 2) (at 114.3 123.698 90)
       (effects (font (size 1.27 1.27)) hide)
@@
   (symbol (lib_id "Device:R") (at 97.79 116.84 90) (unit 1)
     (in_bom yes) (on_board yes)
-    (property "Reference" "R29" (id 0) (at 97.79 122.0978 90))
-    (property "Value" "R" (id 1) (at 97.79 119.7864 90))
+    (property "Reference" "R705" (id 0) (at 97.79 122.0978 90))
+    (property "Value" "10k" (id 1) (at 97.79 119.7864 90))
     (property "Footprint" "Resistor_SMD:R_0603_1608Metric" (id 2) (at 97.79 118.618 90)
       (effects (font (size 1.27 1.27)) hide)
@@
   (symbol (lib_id "Device:R") (at 187.96 121.92 90) (unit 1)
     (in_bom yes) (on_board yes)
-    (property "Reference" "R32" (id 0) (at 187.96 127.1778 90))
-    (property "Value" "R" (id 1) (at 187.96 124.8664 90))
+    (property "Reference" "R708" (id 0) (at 187.96 127.1778 90))
+    (property "Value" "68k" (id 1) (at 187.96 124.8664 90))
     (property "Footprint" "Resistor_SMD:R_0603_1608Metric" (id 2) (at 187.96 123.698 90)
       (effects (font (size 1.27 1.27)) hide)
@@
   (symbol (lib_id "Device:R") (at 171.45 116.84 90) (unit 1)
     (in_bom yes) (on_board yes)
-    (property "Reference" "R30" (id 0) (at 171.45 122.0978 90))
-    (property "Value" "R" (id 1) (at 171.45 119.7864 90))
+    (property "Reference" "R706" (id 0) (at 171.45 122.0978 90))
+    (property "Value" "10k" (id 1) (at 171.45 119.7864 90))
     (property "Footprint" "Resistor_SMD:R_0603_1608Metric" (id 2) (at 171.45 118.618 90)
       (effects (font (size 1.27 1.27)) hide)
@@
   (symbol (lib_id "Jumper:Jumper_3_Open") (at 151.13 161.29 0) (unit 1)
     (in_bom yes) (on_board yes) (fields_autoplaced)
-    (property "Reference" "JP8" (id 0) (at 151.13 154.94 0))
-    (property "Value" "Jumper_3_Open" (id 1) (at 151.13 157.48 0))
+    (property "Reference" "JP701" (id 0) (at 151.13 154.94 0))
+    (property "Value" "DAC AMP" (id 1) (at 151.13 157.48 0))
     (property "Footprint" "Connector_PinHeader_2.54mm:PinHeader_1x03_P2.54mm_Vertical" (id 2) (at 151.13 161.29 0)
       (effects (font (size 1.27 1.27)) hide)
@@
   (symbol (lib_id "power:VDC") (at 160.02 161.29 270) (unit 1)
     (in_bom yes) (on_board yes) (fields_autoplaced)
-    (property "Reference" "#PWR0125" (id 0) (at 157.48 161.29 0)
+    (property "Reference" "#PWR0702" (id 0) (at 157.48 161.29 0)
       (effects (font (size 1.27 1.27)) hide)
     )
@@
   (symbol (lib_id "power:GND") (at 151.13 187.96 0) (unit 1)
     (in_bom yes) (on_board yes) (fields_autoplaced)
-    (property "Reference" "#PWR0126" (id 0) (at 151.13 194.31 0)
+    (property "Reference" "#PWR0703" (id 0) (at 151.13 194.31 0)
       (effects (font (size 1.27 1.27)) hide)
     )
@@
   (symbol (lib_id "power:PWR_FLAG") (at 151.13 167.64 90) (unit 1)
     (in_bom yes) (on_board yes) (fields_autoplaced)
-    (property "Reference" "#FLG06" (id 0) (at 149.225 167.64 0)
+    (property "Reference" "#FLG0701" (id 0) (at 149.225 167.64 0)
       (effects (font (size 1.27 1.27)) hide)
     )
@@
   (symbol (lib_id "power:VCC") (at 142.24 161.29 90) (unit 1)
     (in_bom yes) (on_board yes) (fields_autoplaced)
-    (property "Reference" "#PWR0124" (id 0) (at 146.05 161.29 0)
+    (property "Reference" "#PWR0701" (id 0) (at 146.05 161.29 0)
       (effects (font (size 1.27 1.27)) hide)
     )
@@
   (symbol (lib_id "power:GND") (at 165.1 187.96 0) (unit 1)
     (in_bom yes) (on_board yes) (fields_autoplaced)
-    (property "Reference" "#PWR0127" (id 0) (at 165.1 194.31 0)
-      (effects (font (size 1.27 1.27)) hide)
-    )
+    (property "Reference" "#PWR0704" (id 0) (at 165.1 194.31 0)
+      (effects (font (size 1.27 1.27)) hide)
+    )
