File: AMP_offset.kicad_sch (KiCad schematic)
At the start: 13 parts, among them U25 PDS1-M, U26 Opamp_Dual, U27 MCP4725xxx-xCH

Commit message: layout
Parts:
- C2303: renamed from C69; value C -> 680n
- JP2301: renamed from JP15; value Jumper_3_Open -> DDS AMP
- R2301: renamed from R95; value 5k -> 4k7
- R2302: renamed from R96; value 40k -> 39k
- U2301: renamed from U25; footprint (none) -> PDS1:PSD1
- renumbered C67 to C2301, C68 to C2302, C70 to C2304, C71 to C2305, R97 to R2303, R98 to R2304, U26 to U2302, U27 to U2303
Other:
- moved on the sheet: C2303, R2301, R2302, R2303, U2302A
