File: Battery.kicad_sch (KiCad schematic)
At the start: 19 parts, among them J15 BAT, Q1 Q_NPN_BCE, Q2 Q_PNP_BCE, U2 INA219AxDCN, U3 ISO1540, U4 MCP4725xxx-xCH, U5 Opamp_Dual

Commit message: layout
Parts:
- added C508, C509: 100n, Capacitor_SMD:C_0603_1608Metric, symbol Device:C
- C203: renamed from C3; value 100n -> 1u; footprint Capacitor_SMD:C_0603_1608Metric -> Capacitor_SMD:C_0805_2012Metric
- C204: renamed from C4; value 100n -> 1u; footprint Capacitor_SMD:C_0603_1608Metric -> Capacitor_SMD:C_0805_2012Metric
- renumbered C1 to C201, C2 to C202, C5 to C205, C6 to C206, J15 to J201, PS1 to PS201, Q1 to Q201, Q2 to Q202, R3 to R201, R4 to R202, R5 to R203, R6 to R204, R7 to R205, U2 to U201, U3 to U202, U4 to U203, U5 to U204
Connections:
- net +5VD: now also C508.1, C509.1
- net BAT+: now also U204.6 (-); no longer U204.2 (-)
- net GNDD: now also C508.2, C509.2
- net SCL_: now reaches R202.2, U201.5 (SCL), U202.6 (SCL2), U203.5 (SCL)
- net SCL_: no longer U201.7 (A0), U201.8 (A1)
- net SDA_: now reaches R201.2, U201.6 (SDA), U202.7 (SDA2), U203.4 (SDA)
- net SDA_: now also U201.7 (A0), U201.8 (A1)
- net BAT+_: now reaches Q201.3 (E), Q202.2 (C), R203.1, R205.1
- net at U203.1 (VOUT): now also U204.5 (+); no longer U204.3 (+)
- net at Q201.1 (B), Q202.1 (B): now also U204.7; no longer U204.1
Other:
- moved on the sheet: C202, C203, C204, U204A, U204B, U204C
