File: CAN.kicad_sch (KiCad schematic)
At the start: 12 parts, among them J23 CAN, U18 TJA1051T-3, U19 MCP2515-xSO, Y2 Crystal

Commit message: layout
Parts:
- removed J23: CAN, Connector_PinHeader_2.54mm:PinHeader_1x03_P2.54mm_Vertical, symbol Connector:Conn_01x03_Female
- removed JP13: CAN_term, Connector_PinHeader_2.54mm:PinHeader_1x03_P2.54mm_Vertical, symbol Jumper:Jumper_3_Open
- Y1301: renamed from Y2; value Crystal -> 8MHz; footprint Crystal:Crystal_SMD_HC49-SD -> Crystal:Crystal_SMD_5032-2Pin_5.0x3.2mm
- renumbered C45 to C1301, C46 to C1302, C47 to C1303, C48 to C1304, JP12 to JP1301, R74 to R1301, R75 to R1302, U18 to U1301, U19 to U1302
Connections:
- net CANL: now reaches U1301.6 (CANL)
- net CANL: now also R1301.1
- net CANH: now reaches U1301.7 (CANH)
- net CANH: now also R1301.2; no longer R1301.1
- no-connect marks 9 -> 8
Other:
- moved on the sheet: R1301
