File: Current.kicad_sch (KiCad schematic)
At the start: 6 parts

Commit message: layout
Parts:
- C1901: renamed from C59; value (none) -> 100n; footprint (none) -> Capacitor_SMD:C_0603_1608Metric
- C1902: renamed from C60; value (none) -> 100n; footprint (none) -> Capacitor_SMD:C_0603_1608Metric
- R1901: renamed from R81; value (none) -> 10R; footprint (none) -> Resistor_SMD:R_0603_1608Metric
- R1902: renamed from R82; value (none) -> 100R; footprint (none) -> Resistor_SMD:R_2512_6332Metric
- R1903: renamed from R83; value (none) -> 10R; footprint (none) -> Resistor_SMD:R_0603_1608Metric
- U1901: renamed from U23; value (none) -> INA219AxDCN; footprint (none) -> Package_TO_SOT_SMD:SOT-23-8
Changed lines of the file:
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@@
   (symbol (lib_id "Device:R") (at 99.06 104.14 0) (unit 1)
     (in_bom yes) (on_board yes)
-    (property "Reference" "R82" (id 0) (at 100.838 102.9716 0)
+    (property "Reference" "R1902" (id 0) (at 100.838 102.9716 0)
       (effects (font (size 1.27 1.27)) (justify left))
     )
-    (property "Value" "" (id 1) (at 100.838 105.283 0)
+    (property "Value" "100R" (id 1) (at 100.838 105.283 0)
       (effects (font (size 1.27 1.27)) (justify left))
     )
-    (property "Footprint" "" (id 2) (at 97.282 104.14 90)
+    (property "Footprint" "Resistor_SMD:R_2512_6332Metric" (id 2) (at 97.282 104.14 90)
       (effects (font (size 1.27 1.27)) hide)
     )
@@
   (symbol (lib_id "power:+3V3") (at 166.37 177.8 0) (unit 1)
     (in_bom yes) (on_board yes)
-    (property "Reference" "#PWR?" (id 0) (at 166.37 181.61 0)
+    (property "Reference" "#PWR01903" (id 0) (at 166.37 181.61 0)
       (effects (font (size 1.27 1.27)) hide)
     )
-    (property "Value" "" (id 1) (at 166.751 173.4058 0))
+    (property "Value" "+3V3" (id 1) (at 166.751 173.4058 0))
     (property "Footprint" "" (id 2) (at 166.37 177.8 0)
       (effects (font (size 1.27 1.27)) hide)
@@
   (symbol (lib_id "power:GND") (at 166.37 187.96 0) (unit 1)
     (in_bom yes) (on_board yes)
-    (property "Reference" "#PWR?" (id 0) (at 166.37 194.31 0)
+    (property "Reference" "#PWR01904" (id 0) (at 166.37 194.31 0)
       (effects (font (size 1.27 1.27)) hide)
     )
-    (property "Value" "" (id 1) (at 166.497 192.3542 0))
+    (property "Value" "GND" (id 1) (at 166.497 192.3542 0))
     (property "Footprint" "" (id 2) (at 166.37 187.96 0)
       (effects (font (size 1.27 1.27)) hide)
@@
   (symbol (lib_id "power:GND") (at 148.59 116.84 0) (unit 1)
     (in_bom yes) (on_board yes)
-    (property "Reference" "#PWR?" (id 0) (at 148.59 123.19 0)
+    (property "Reference" "#PWR01902" (id 0) (at 148.59 123.19 0)
       (effects (font (size 1.27 1.27)) hide)
     )
-    (property "Value" "" (id 1) (at 148.717 121.2342 0))
+    (property "Value" "GND" (id 1) (at 148.717 121.2342 0))
     (property "Footprint" "" (id 2) (at 148.59 116.84 0)
       (effects (font (size 1.27 1.27)) hide)
@@
   (symbol (lib_id "Analog_ADC:INA219AxDCN") (at 148.59 104.14 0) (unit 1)
     (in_bom yes) (on_board yes) (fields_autoplaced)
-    (property "Reference" "U23" (id 0) (at 150.6094 91.44 0)
+    (property "Reference" "U1901" (id 0) (at 150.6094 91.44 0)
       (effects (font (size 1.27 1.27)) (justify left))
     )
-    (property "Value" "" (id 1) (at 150.6094 93.98 0)
+    (property "Value" "INA219AxDCN" (id 1) (at 150.6094 93.98 0)
       (effects (font (size 1.27 1.27)) (justify left))
     )
-    (property "Footprint" "" (id 2) (at 165.1 113.03 0)
+    (property "Footprint" "Package_TO_SOT_SMD:SOT-23-8" (id 2) (at 165.1 113.03 0)
       (effects (font (size 1.27 1.27)) hide)
     )
@@
   (symbol (lib_id "Device:C") (at 166.37 182.88 0) (unit 1)
     (in_bom yes) (on_board yes)
-    (property "Reference" "C60" (id 0) (at 169.291 181.7116 0)
+    (property "Reference" "C1902" (id 0) (at 169.291 181.7116 0)
       (effects (font (size 1.27 1.27)) (justify left))
     )
-    (property "Value" "" (id 1) (at 169.291 184.023 0)
+    (property "Value" "100n" (id 1) (at 169.291 184.023 0)
       (effects (font (size 1.27 1.27)) (justify left))
     )
-    (property "Footprint" "" (id 2) (at 167.3352 186.69 0)
+    (property "Footprint" "Capacitor_SMD:C_0603_1608Metric" (id 2) (at 167.3352 186.69 0)
       (effects (font (size 1.27 1.27)) hide)
     )
@@
   (symbol (lib_id "Device:C") (at 119.38 104.14 0) (unit 1)
     (in_bom yes) (on_board yes) (fields_autoplaced)
-    (property "Reference" "C59" (id 0) (at 123.19 102.8699 0)
+    (property "Reference" "C1901" (id 0) (at 123.19 102.8699 0)
       (effects (font (size 1.27 1.27)) (justify left))
     )
-    (property "Value" "" (id 1) (at 123.19 105.4099 0)
+    (property "Value" "100n" (id 1) (at 123.19 105.4099 0)
       (effects (font (size 1.27 1.27)) (justify left))
     )
-    (property "Footprint" "" (id 2) (at 120.3452 107.95 0)
+    (property "Footprint" "Capacitor_SMD:C_0603_1608Metric" (id 2) (at 120.3452 107.95 0)
       (effects (font (size 1.27 1.27)) hide)
     )
@@
   (symbol (lib_id "Device:R") (at 113.03 109.22 90) (unit 1)
     (in_bom yes) (on_board yes) (fields_autoplaced)
-    (property "Reference" "R83" (id 0) (at 113.03 102.87 90))
-    (property "Value" "" (id 1) (at 113.03 105.41 90))
-    (property "Footprint" "" (id 2) (at 113.03 110.998 90)
+    (property "Reference" "R1903" (id 0) (at 113.03 102.87 90))
+    (property "Value" "10R" (id 1) (at 113.03 105.41 90))
+    (property "Footprint" "Resistor_SMD:R_0603_1608Metric" (id 2) (at 113.03 110.998 90)
       (effects (font (size 1.27 1.27)) hide)
     )
@@
   (symbol (lib_id "power:+3V3") (at 148.59 91.44 0) (unit 1)
     (in_bom yes) (on_board yes)
-    (property "Reference" "#PWR?" (id 0) (at 148.59 95.25 0)
+    (property "Reference" "#PWR01901" (id 0) (at 148.59 95.25 0)
       (effects (font (size 1.27 1.27)) hide)
     )
-    (property "Value" "" (id 1) (at 148.971 87.0458 0))
+    (property "Value" "+3V3" (id 1) (at 148.971 87.0458 0))
     (property "Footprint" "" (id 2) (at 148.59 91.44 0)
       (effects (font (size 1.27 1.27)) hide)
@@
   (symbol (lib_id "Device:R") (at 113.03 99.06 90) (unit 1)
     (in_bom yes) (on_board yes) (fields_autoplaced)
-    (property "Reference" "R81" (id 0) (at 113.03 92.71 90))
-    (property "Value" "" (id 1) (at 113.03 95.25 90))
-    (property "Footprint" "" (id 2) (at 113.03 100.838 90)
+    (property "Reference" "R1901" (id 0) (at 113.03 92.71 90))
+    (property "Value" "10R" (id 1) (at 113.03 95.25 90))
+    (property "Footprint" "Resistor_SMD:R_0603_1608Metric" (id 2) (at 113.03 100.838 90)
       (effects (font (size 1.27 1.27)) hide)
     )
