File: DAC.kicad_sch (KiCad schematic)
At the start: 4 parts, among them U16 MCP4728

Commit message: layout
Parts:
- removed C34: 10u, Capacitor_SMD:C_0805_2012Metric, symbol Device:C
- renumbered C35 to C901, R33 to R901, U16 to U901
Changed lines of the file:
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@@
-    (stroke (width 0) (type default) (color 0 0 0 0))
-  )
-  (wire (pts (xy 152.4 176.53) (xy 152.4 175.26))
     (stroke (width 0) (type default) (color 0 0 0 0))
   )
@@
   )
   (wire (pts (xy 158.75 106.68) (xy 154.94 106.68))
-    (stroke (width 0) (type default) (color 0 0 0 0))
-  )
-  (wire (pts (xy 152.4 184.15) (xy 152.4 185.42))
     (stroke (width 0) (type default) (color 0 0 0 0))
   )
@@
   (symbol (lib_id "power:+3V3") (at 139.7 90.17 0) (unit 1)
     (in_bom yes) (on_board yes)
-    (property "Reference" "#PWR0136" (id 0) (at 139.7 93.98 0)
+    (property "Reference" "#PWR0901" (id 0) (at 139.7 93.98 0)
       (effects (font (size 1.27 1.27)) hide)
     )
@@
   (symbol (lib_id "power:GND") (at 139.7 115.57 0) (unit 1)
     (in_bom yes) (on_board yes)
-    (property "Reference" "#PWR0137" (id 0) (at 139.7 121.92 0)
+    (property "Reference" "#PWR0902" (id 0) (at 139.7 121.92 0)
       (effects (font (size 1.27 1.27)) hide)
     )
@@
   (symbol (lib_id "power:GND") (at 165.1 185.42 0) (unit 1)
     (in_bom yes) (on_board yes)
-    (property "Reference" "#PWR0142" (id 0) (at 165.1 191.77 0)
+    (property "Reference" "#PWR0905" (id 0) (at 165.1 191.77 0)
       (effects (font (size 1.27 1.27)) hide)
     )
@@
   (symbol (lib_id "power:+3V3") (at 165.1 175.26 0) (unit 1)
     (in_bom yes) (on_board yes)
-    (property "Reference" "#PWR0140" (id 0) (at 165.1 179.07 0)
+    (property "Reference" "#PWR0904" (id 0) (at 165.1 179.07 0)
       (effects (font (size 1.27 1.27)) hide)
     )
@@
   (symbol (lib_id "Device:C") (at 165.1 180.34 0) (unit 1)
     (in_bom yes) (on_board yes)
-    (property "Reference" "C35" (id 0) (at 168.021 179.1716 0)
+    (property "Reference" "C901" (id 0) (at 168.021 179.1716 0)
       (effects (font (size 1.27 1.27)) (justify left))
     )
@@
   (symbol (lib_id "Device:R") (at 113.03 111.76 0) (unit 1)
     (in_bom yes) (on_board yes)
-    (property "Reference" "R33" (id 0) (at 114.808 110.5916 0)
+    (property "Reference" "R901" (id 0) (at 114.808 110.5916 0)
       (effects (font (size 1.27 1.27)) (justify left))
     )
@@
   (symbol (lib_id "power:GND") (at 113.03 118.11 0) (unit 1)
     (in_bom yes) (on_board yes)
-    (property "Reference" "#PWR0138" (id 0) (at 113.03 124.46 0)
+    (property "Reference" "#PWR0903" (id 0) (at 113.03 124.46 0)
       (effects (font (size 1.27 1.27)) hide)
     )
@@
   (symbol (lib_id "Analog_DAC:MCP4728") (at 139.7 101.6 0) (unit 1)
     (in_bom yes) (on_board yes)
-    (property "Reference" "U16" (id 0) (at 139.7 77.47 0))
+    (property "Reference" "U901" (id 0) (at 139.7 77.47 0))
     (property "Value" "MCP4728" (id 1) (at 139.7 80.01 0))
     (property "Footprint" "Package_SO:MSOP-10_3x3mm_P0.5mm" (id 2) (at 139.7 116.84 0)
@@
     (pin "9")
   )
-  (symbol (lib_id "power:GND") (at 152.4 185.42 0) (unit 1)
-    (in_bom yes) (on_board yes)
-    (property "Reference" "#PWR0141" (id 0) (at 152.4 191.77 0)
-      (effects (font (size 1.27 1.27)) hide)
-    )
-    (property "Value" "GND" (id 1) (at 152.527 189.8142 0))
-    (property "Footprint" "" (id 2) (at 152.4 185.42 0)
-      (effects (font (size 1.27 1.27)) hide)
-    )
-    (property "Datasheet" "" (id 3) (at 152.4 185.42 0)
-      (effects (font (size 1.27 1.27)) hide)
-    )
-    (pin "1")
-  )
-  (symbol (lib_id "power:+3V3") (at 152.4 175.26 0) (unit 1)
-    (in_bom yes) (on_board yes)
-    (property "Reference" "#PWR0139" (id 0) (at 152.4 179.07 0)
-      (effects (font (size 1.27 1.27)) hide)
-    )
-    (property "Value" "+3V3" (id 1) (at 152.781 170.8658 0))
-    (property "Footprint" "" (id 2) (at 152.4 175.26 0)
-      (effects (font (size 1.27 1.27)) hide)
-    )
-    (property "Datasheet" "" (id 3) (at 152.4 175.26 0)
-      (effects (font (size 1.27 1.27)) hide)
-    )
-    (pin "1")
-  )
-  (symbol (lib_id "Device:C") (at 152.4 180.34 0) (unit 1)
-    (in_bom yes) (on_board yes)
-    (property "Reference" "C34" (id 0) (at 155.321 179.1716 0)
-      (effects (font (size 1.27 1.27)) (justify left))
-    )
-    (property "Value" "10u" (id 1) (at 155.321 181.483 0)
-      (effects (font (size 1.27 1.27)) (justify left))
-    )
-    (property "Footprint" "Capacitor_SMD:C_0805_2012Metric" (id 2) (at 153.3652 184.15 0)
-      (effects (font (size 1.27 1.27)) hide)
-    )
-    (property "Datasheet" "~" (id 3) (at 152.4 180.34 0)
-      (effects (font (size 1.27 1.27)) hide)
-    )
-    (pin "1")
-    (pin "2")
-  )
 )
