File: DDS.kicad_sch (KiCad schematic)
At the start: 7 parts, among them U20 AD9833xRM, X1 XO32

Commit message: layout
Parts:
- removed C52: 100n, Capacitor_SMD:C_0603_1608Metric, symbol Device:C
- renumbered C49 to C1401, C50 to C1402, C51 to C1403, C53 to C1404, U20 to U1401, X1 to X1401
Changed lines of the file:
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@@
   )
   (no_connect (at 100.33 109.22))
-  (wire (pts (xy 153.67 186.69) (xy 153.67 185.42))
-    (stroke (width 0) (type default) (color 0 0 0 0))
-  )
   (wire (pts (xy 143.51 118.11) (xy 143.51 116.84))
     (stroke (width 0) (type default) (color 0 0 0 0))
@@
   )
   (wire (pts (xy 148.59 91.44) (xy 148.59 90.17))
-    (stroke (width 0) (type default) (color 0 0 0 0))
-  )
-  (wire (pts (xy 153.67 177.8) (xy 153.67 176.53))
     (stroke (width 0) (type default) (color 0 0 0 0))
   )
@@
   (symbol (lib_id "Interface:AD9833xRM") (at 146.05 104.14 0) (unit 1)
     (in_bom yes) (on_board yes)
-    (property "Reference" "U20" (id 0) (at 144.78 72.39 0)
+    (property "Reference" "U1401" (id 0) (at 144.78 72.39 0)
       (effects (font (size 1.27 1.27)) (justify left))
     )
@@
   (symbol (lib_id "power:+3V3") (at 148.59 90.17 0) (unit 1)
     (in_bom yes) (on_board yes)
-    (property "Reference" "#PWR0199" (id 0) (at 148.59 93.98 0)
+    (property "Reference" "#PWR01402" (id 0) (at 148.59 93.98 0)
       (effects (font (size 1.27 1.27)) hide)
     )
@@
   (symbol (lib_id "power:GND") (at 143.51 118.11 0) (unit 1)
     (in_bom yes) (on_board yes)
-    (property "Reference" "#PWR0203" (id 0) (at 143.51 124.46 0)
+    (property "Reference" "#PWR01406" (id 0) (at 143.51 124.46 0)
       (effects (font (size 1.27 1.27)) hide)
     )
@@
   (symbol (lib_id "Device:C") (at 127 85.09 0) (unit 1)
     (in_bom yes) (on_board yes)
-    (property "Reference" "C49" (id 0) (at 129.921 83.9216 0)
+    (property "Reference" "C1401" (id 0) (at 129.921 83.9216 0)
       (effects (font (size 1.27 1.27)) (justify left))
     )
@@
   (symbol (lib_id "power:GND") (at 148.59 118.11 0) (unit 1)
     (in_bom yes) (on_board yes)
-    (property "Reference" "#PWR0204" (id 0) (at 148.59 124.46 0)
+    (property "Reference" "#PWR01407" (id 0) (at 148.59 124.46 0)
       (effects (font (size 1.27 1.27)) hide)
     )
@@
   (symbol (lib_id "Device:C") (at 166.37 96.52 0) (unit 1)
     (in_bom yes) (on_board yes)
-    (property "Reference" "C50" (id 0) (at 169.291 95.3516 0)
+    (property "Reference" "C1402" (id 0) (at 169.291 95.3516 0)
       (effects (font (size 1.27 1.27)) (justify left))
     )
@@
   (symbol (lib_id "power:GND") (at 127 90.17 0) (unit 1)
     (in_bom yes) (on_board yes)
-    (property "Reference" "#PWR0198" (id 0) (at 127 96.52 0)
+    (property "Reference" "#PWR01401" (id 0) (at 127 96.52 0)
       (effects (font (size 1.27 1.27)) hide)
     )
@@
   (symbol (lib_id "power:+3V3") (at 166.37 90.17 0) (unit 1)
     (in_bom yes) (on_board yes)
-    (property "Reference" "#PWR0200" (id 0) (at 166.37 93.98 0)
+    (property "Reference" "#PWR01403" (id 0) (at 166.37 93.98 0)
       (effects (font (size 1.27 1.27)) hide)
     )
@@
   (symbol (lib_id "Device:C") (at 165.1 181.61 0) (unit 1)
     (in_bom yes) (on_board yes)
-    (property "Reference" "C53" (id 0) (at 168.021 180.4416 0)
+    (property "Reference" "C1404" (id 0) (at 168.021 180.4416 0)
       (effects (font (size 1.27 1.27)) (justify left))
     )
@@
   (symbol (lib_id "power:GND") (at 165.1 186.69 0) (unit 1)
     (in_bom yes) (on_board yes)
-    (property "Reference" "#PWR0209" (id 0) (at 165.1 193.04 0)
+    (property "Reference" "#PWR01410" (id 0) (at 165.1 193.04 0)
       (effects (font (size 1.27 1.27)) hide)
     )
@@
   (symbol (lib_id "power:+3V3") (at 165.1 176.53 0) (unit 1)
     (in_bom yes) (on_board yes)
-    (property "Reference" "#PWR0207" (id 0) (at 165.1 180.34 0)
+    (property "Reference" "#PWR01409" (id 0) (at 165.1 180.34 0)
       (effects (font (size 1.27 1.27)) hide)
     )
@@
   (symbol (lib_id "Device:C") (at 166.37 113.03 0) (unit 1)
     (in_bom yes) (on_board yes) (fields_autoplaced)
-    (property "Reference" "C51" (id 0) (at 170.18 111.7599 0)
+    (property "Reference" "C1403" (id 0) (at 170.18 111.7599 0)
       (effects (font (size 1.27 1.27)) (justify left))
     )
@@
   (symbol (lib_id "power:+3V3") (at 107.95 100.33 0) (unit 1)
     (in_bom yes) (on_board yes)
-    (property "Reference" "#PWR0201" (id 0) (at 107.95 104.14 0)
+    (property "Reference" "#PWR01404" (id 0) (at 107.95 104.14 0)
       (effects (font (size 1.27 1.27)) hide)
     )
@@
   (symbol (lib_id "power:GND") (at 166.37 118.11 0) (unit 1)
     (in_bom yes) (on_board yes)
-    (property "Reference" "#PWR0205" (id 0) (at 166.37 124.46 0)
+    (property "Reference" "#PWR01408" (id 0) (at 166.37 124.46 0)
       (effects (font (size 1.27 1.27)) hide)
     )
@@
     (pin "1")
   )
-  (symbol (lib_id "power:+3V3") (at 153.67 176.53 0) (unit 1)
-    (in_bom yes) (on_board yes)
-    (property "Reference" "#PWR0206" (id 0) (at 153.67 180.34 0)
-      (effects (font (size 1.27 1.27)) hide)
-    )
-    (property "Value" "+3V3" (id 1) (at 154.051 172.1358 0))
-    (property "Footprint" "" (id 2) (at 153.67 176.53 0)
-      (effects (font (size 1.27 1.27)) hide)
-    )
-    (property "Datasheet" "" (id 3) (at 153.67 176.53 0)
-      (effects (font (size 1.27 1.27)) hide)
-    )
-    (pin "1")
-  )
   (symbol (lib_id "power:PWR_FLAG") (at 143.51 80.01 270) (unit 1)
     (in_bom yes) (on_board yes) (fields_autoplaced)
-    (property "Reference" "#FLG08" (id 0) (at 145.415 80.01 0)
+    (property "Reference" "#FLG01401" (id 0) (at 145.415 80.01 0)
       (effects (font (size 1.27 1.27)) hide)
     )
@@
     )
     (property "Datasheet" "~" (id 3) (at 143.51 80.01 0)
-      (effects (font (size 1.27 1.27)) hide)
-    )
-    (pin "1")
-  )
-  (symbol (lib_id "Device:C") (at 153.67 181.61 0) (unit 1)
-    (in_bom yes) (on_board yes)
-    (property "Reference" "C52" (id 0) (at 156.591 180.4416 0)
-      (effects (font (size 1.27 1.27)) (justify left))
-    )
-    (property "Value" "100n" (id 1) (at 156.591 182.753 0)
-      (effects (font (size 1.27 1.27)) (justify left))
-    )
-    (property "Footprint" "Capacitor_SMD:C_0603_1608Metric" (id 2) (at 154.6352 185.42 0)
-      (effects (font (size 1.27 1.27)) hide)
-    )
-    (property "Datasheet" "~" (id 3) (at 153.67 181.61 0)
-      (effects (font (size 1.27 1.27)) hide)
-    )
-    (pin "1")
-    (pin "2")
-  )
-  (symbol (lib_id "power:GND") (at 153.67 186.69 0) (unit 1)
-    (in_bom yes) (on_board yes)
-    (property "Reference" "#PWR0208" (id 0) (at 153.67 193.04 0)
-      (effects (font (size 1.27 1.27)) hide)
-    )
-    (property "Value" "GND" (id 1) (at 153.797 191.0842 0))
-    (property "Footprint" "" (id 2) (at 153.67 186.69 0)
-      (effects (font (size 1.27 1.27)) hide)
-    )
-    (property "Datasheet" "" (id 3) (at 153.67 186.69 0)
       (effects (font (size 1.27 1.27)) hide)
     )
@@
   (symbol (lib_id "Oscillator:XO32") (at 107.95 109.22 0) (unit 1)
     (in_bom yes) (on_board yes) (fields_autoplaced)
-    (property "Reference" "X1" (id 0) (at 116.84 104.8893 0))
+    (property "Reference" "X1401" (id 0) (at 116.84 104.8893 0))
     (property "Value" "XO32" (id 1) (at 116.84 107.4293 0))
     (property "Footprint" "Oscillator:Oscillator_SMD_EuroQuartz_XO32-4Pin_3.2x2.5mm_HandSoldering" (id 2) (at 125.73 118.11 0)
@@
   (symbol (lib_id "power:GND") (at 107.95 118.11 0) (unit 1)
     (in_bom yes) (on_board yes)
-    (property "Reference" "#PWR0202" (id 0) (at 107.95 124.46 0)
-      (effects (font (size 1.27 1.27)) hide)
-    )
+    (property "Reference" "#PWR01405" (id 0) (at 107.95 124.46 0)
+      (effects (font (size 1.27 1.27)) hide)
+    )
