File: EEPROM.kicad_sch (KiCad schematic)
At the start: 2 parts, among them U22 24LC32

Commit message: layout
Parts:
- renumbered C58 to C1801, U22 to U1801
Changed lines of the file:
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@@
   (symbol (lib_id "power:+3V3") (at 146.05 86.36 0) (unit 1)
     (in_bom yes) (on_board yes) (fields_autoplaced)
-    (property "Reference" "#PWR0230" (id 0) (at 146.05 90.17 0)
+    (property "Reference" "#PWR01801" (id 0) (at 146.05 90.17 0)
       (effects (font (size 1.27 1.27)) hide)
     )
@@
   (symbol (lib_id "Device:C") (at 165.1 180.34 0) (unit 1)
     (in_bom yes) (on_board yes) (fields_autoplaced)
-    (property "Reference" "C58" (id 0) (at 168.91 179.0699 0)
+    (property "Reference" "C1801" (id 0) (at 168.91 179.0699 0)
       (effects (font (size 1.27 1.27)) (justify left))
     )
@@
   (symbol (lib_id "power:GND") (at 165.1 186.69 0) (unit 1)
     (in_bom yes) (on_board yes) (fields_autoplaced)
-    (property "Reference" "#PWR0234" (id 0) (at 165.1 193.04 0)
+    (property "Reference" "#PWR01805" (id 0) (at 165.1 193.04 0)
       (effects (font (size 1.27 1.27)) hide)
     )
@@
   (symbol (lib_id "power:+3V3") (at 165.1 173.99 0) (unit 1)
     (in_bom yes) (on_board yes) (fields_autoplaced)
-    (property "Reference" "#PWR0233" (id 0) (at 165.1 177.8 0)
+    (property "Reference" "#PWR01804" (id 0) (at 165.1 177.8 0)
       (effects (font (size 1.27 1.27)) hide)
     )
@@
   (symbol (lib_id "Memory_EEPROM:24LC32") (at 146.05 97.79 0) (unit 1)
     (in_bom yes) (on_board yes) (fields_autoplaced)
-    (property "Reference" "U22" (id 0) (at 148.0694 87.63 0)
+    (property "Reference" "U1801" (id 0) (at 148.0694 87.63 0)
       (effects (font (size 1.27 1.27)) (justify left))
     )
@@
   (symbol (lib_id "power:GND") (at 132.08 113.03 0) (unit 1)
     (in_bom yes) (on_board yes) (fields_autoplaced)
-    (property "Reference" "#PWR0231" (id 0) (at 132.08 119.38 0)
+    (property "Reference" "#PWR01802" (id 0) (at 132.08 119.38 0)
       (effects (font (size 1.27 1.27)) hide)
     )
@@
   (symbol (lib_id "power:GND") (at 146.05 113.03 0) (unit 1)
     (in_bom yes) (on_board yes) (fields_autoplaced)
-    (property "Reference" "#PWR0232" (id 0) (at 146.05 119.38 0)
+    (property "Reference" "#PWR01803" (id 0) (at 146.05 119.38 0)
       (effects (font (size 1.27 1.27)) hide)
     )
