File: ESP8266.kicad_sch (KiCad schematic)
At the start: 6 parts, among them J24 ESP8266

Commit message: layout
Parts:
- R1501: renamed from R76; footprint Resistor_SMD:R_0201_0603Metric -> Resistor_SMD:R_0603_1608Metric
- R1502: renamed from R77; footprint Resistor_SMD:R_0201_0603Metric -> Resistor_SMD:R_0603_1608Metric
- R1503: renamed from R78; footprint Resistor_SMD:R_0201_0603Metric -> Resistor_SMD:R_0603_1608Metric
- R1504: renamed from R79; footprint Resistor_SMD:R_0201_0603Metric -> Resistor_SMD:R_0603_1608Metric
- renumbered C54 to C1501, J24 to J1501
Changed lines of the file:
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@@
   (symbol (lib_id "Device:C") (at 163.83 181.61 0) (unit 1)
     (in_bom yes) (on_board yes) (fields_autoplaced)
-    (property "Reference" "C54" (id 0) (at 167.64 180.3399 0)
+    (property "Reference" "C1501" (id 0) (at 167.64 180.3399 0)
       (effects (font (size 1.27 1.27)) (justify left))
     )
@@
   (symbol (lib_id "power:GND") (at 163.83 91.44 0) (unit 1)
     (in_bom yes) (on_board yes) (fields_autoplaced)
-    (property "Reference" "#PWR0212" (id 0) (at 163.83 97.79 0)
+    (property "Reference" "#PWR01503" (id 0) (at 163.83 97.79 0)
       (effects (font (size 1.27 1.27)) hide)
     )
@@
   (symbol (lib_id "power:+3V3") (at 181.61 114.3 270) (unit 1)
     (in_bom yes) (on_board yes) (fields_autoplaced)
-    (property "Reference" "#PWR0214" (id 0) (at 177.8 114.3 0)
+    (property "Reference" "#PWR01505" (id 0) (at 177.8 114.3 0)
       (effects (font (size 1.27 1.27)) hide)
     )
@@
   (symbol (lib_id "power:GND") (at 163.83 189.23 0) (unit 1)
     (in_bom yes) (on_board yes) (fields_autoplaced)
-    (property "Reference" "#PWR0216" (id 0) (at 163.83 195.58 0)
+    (property "Reference" "#PWR01507" (id 0) (at 163.83 195.58 0)
       (effects (font (size 1.27 1.27)) hide)
     )
@@
   (symbol (lib_id "Device:R") (at 172.72 92.71 0) (unit 1)
     (in_bom yes) (on_board yes) (fields_autoplaced)
-    (property "Reference" "R77" (id 0) (at 175.26 91.4399 0)
+    (property "Reference" "R1502" (id 0) (at 175.26 91.4399 0)
       (effects (font (size 1.27 1.27)) (justify left))
     )
@@
       (effects (font (size 1.27 1.27)) (justify left))
     )
-    (property "Footprint" "Resistor_SMD:R_0201_0603Metric" (id 2) (at 170.942 92.71 90)
+    (property "Footprint" "Resistor_SMD:R_0603_1608Metric" (id 2) (at 170.942 92.71 90)
       (effects (font (size 1.27 1.27)) hide)
     )
@@
   (symbol (lib_id "Device:R") (at 121.92 107.95 0) (unit 1)
     (in_bom yes) (on_board yes) (fields_autoplaced)
-    (property "Reference" "R78" (id 0) (at 124.46 106.6799 0)
+    (property "Reference" "R1503" (id 0) (at 124.46 106.6799 0)
       (effects (font (size 1.27 1.27)) (justify left))
     )
@@
       (effects (font (size 1.27 1.27)) (justify left))
     )
-    (property "Footprint" "Resistor_SMD:R_0201_0603Metric" (id 2) (at 120.142 107.95 90)
+    (property "Footprint" "Resistor_SMD:R_0603_1608Metric" (id 2) (at 120.142 107.95 90)
       (effects (font (size 1.27 1.27)) hide)
     )
@@
   (symbol (lib_id "Device:R") (at 121.92 92.71 0) (unit 1)
     (in_bom yes) (on_board yes) (fields_autoplaced)
-    (property "Reference" "R76" (id 0) (at 124.46 91.4399 0)
+    (property "Reference" "R1501" (id 0) (at 124.46 91.4399 0)
       (effects (font (size 1.27 1.27)) (justify left))
     )
@@
       (effects (font (size 1.27 1.27)) (justify left))
     )
-    (property "Footprint" "Resistor_SMD:R_0201_0603Metric" (id 2) (at 120.142 92.71 90)
+    (property "Footprint" "Resistor_SMD:R_0603_1608Metric" (id 2) (at 120.142 92.71 90)
       (effects (font (size 1.27 1.27)) hide)
     )
@@
   (symbol (lib_id "power:+3V3") (at 181.61 86.36 270) (unit 1)
     (in_bom yes) (on_board yes) (fields_autoplaced)
-    (property "Reference" "#PWR0211" (id 0) (at 177.8 86.36 0)
+    (property "Reference" "#PWR01502" (id 0) (at 177.8 86.36 0)
       (effects (font (size 1.27 1.27)) hide)
     )
@@
   (symbol (lib_id "power:+3V3") (at 163.83 173.99 0) (unit 1)
     (in_bom yes) (on_board yes) (fields_autoplaced)
-    (property "Reference" "#PWR0215" (id 0) (at 163.83 177.8 0)
+    (property "Reference" "#PWR01506" (id 0) (at 163.83 177.8 0)
       (effects (font (size 1.27 1.27)) hide)
     )
@@
   (symbol (lib_id "Device:R") (at 172.72 107.95 0) (unit 1)
     (in_bom yes) (on_board yes) (fields_autoplaced)
-    (property "Reference" "R79" (id 0) (at 175.26 106.6799 0)
+    (property "Reference" "R1504" (id 0) (at 175.26 106.6799 0)
       (effects (font (size 1.27 1.27)) (justify left))
     )
@@
       (effects (font (size 1.27 1.27)) (justify left))
     )
-    (property "Footprint" "Resistor_SMD:R_0201_0603Metric" (id 2) (at 170.942 107.95 90)
+    (property "Footprint" "Resistor_SMD:R_0603_1608Metric" (id 2) (at 170.942 107.95 90)
       (effects (font (size 1.27 1.27)) hide)
     )
@@
   (symbol (lib_id "Connector_Generic:Conn_02x04_Counter_Clockwise") (at 144.78 99.06 0) (unit 1)
     (in_bom yes) (on_board yes) (fields_autoplaced)
-    (property "Reference" "J24" (id 0) (at 146.05 90.17 0))
+    (property "Reference" "J1501" (id 0) (at 146.05 90.17 0))
     (property "Value" "ESP8266" (id 1) (at 146.05 92.71 0))
     (property "Footprint" "Connector_PinHeader_2.54mm:PinHeader_2x04_P2.54mm_Vertical" (id 2) (at 144.78 99.06 0)
@@
   (symbol (lib_id "power:+3V3") (at 115.57 114.3 90) (unit 1)
     (in_bom yes) (on_board yes) (fields_autoplaced)
-    (property "Reference" "#PWR0213" (id 0) (at 119.38 114.3 0)
+    (property "Reference" "#PWR01504" (id 0) (at 119.38 114.3 0)
       (effects (font (size 1.27 1.27)) hide)
     )
@@
   (symbol (lib_id "power:+3V3") (at 115.57 86.36 90) (unit 1)
     (in_bom yes) (on_board yes) (fields_autoplaced)
-    (property "Reference" "#PWR0210" (id 0) (at 119.38 86.36 0)
-      (effects (font (size 1.27 1.27)) hide)
-    )
+    (property "Reference" "#PWR01501" (id 0) (at 119.38 86.36 0)
+      (effects (font (size 1.27 1.27)) hide)
+    )
