File: IO_Expander.kicad_sch (KiCad schematic)
At the start: 3 parts, among them U28 MCP23017_SS

Commit message: layout
Parts:
- renumbered C72 to C2401, R101 to R2401, U28 to U2401
Changed lines of the file:
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@@
   (symbol (lib_id "power:+3V3") (at 114.3 85.09 0) (unit 1)
     (in_bom yes) (on_board yes) (fields_autoplaced)
-    (property "Reference" "#PWR0278" (id 0) (at 114.3 88.9 0)
+    (property "Reference" "#PWR02402" (id 0) (at 114.3 88.9 0)
       (effects (font (size 1.27 1.27)) hide)
     )
@@
   (symbol (lib_id "Interface_Expansion:MCP23017_SS") (at 146.05 102.87 0) (unit 1)
     (in_bom yes) (on_board yes) (fields_autoplaced)
-    (property "Reference" "U28" (id 0) (at 148.0694 74.93 0)
+    (property "Reference" "U2401" (id 0) (at 148.0694 74.93 0)
       (effects (font (size 1.27 1.27)) (justify left))
     )
@@
   (symbol (lib_id "power:GND") (at 125.73 133.35 0) (unit 1)
     (in_bom yes) (on_board yes)
-    (property "Reference" "#PWR0279" (id 0) (at 125.73 139.7 0)
+    (property "Reference" "#PWR02403" (id 0) (at 125.73 139.7 0)
       (effects (font (size 1.27 1.27)) hide)
     )
@@
   (symbol (lib_id "Device:C") (at 165.1 180.34 0) (unit 1)
     (in_bom yes) (on_board yes) (fields_autoplaced)
-    (property "Reference" "C72" (id 0) (at 168.91 179.0699 0)
+    (property "Reference" "C2401" (id 0) (at 168.91 179.0699 0)
       (effects (font (size 1.27 1.27)) (justify left))
     )
@@
   (symbol (lib_id "power:GND") (at 146.05 133.35 0) (unit 1)
     (in_bom yes) (on_board yes)
-    (property "Reference" "#PWR0280" (id 0) (at 146.05 139.7 0)
+    (property "Reference" "#PWR02404" (id 0) (at 146.05 139.7 0)
       (effects (font (size 1.27 1.27)) hide)
     )
@@
   (symbol (lib_id "power:+3V3") (at 146.05 72.39 0) (unit 1)
     (in_bom yes) (on_board yes) (fields_autoplaced)
-    (property "Reference" "#PWR0275" (id 0) (at 146.05 76.2 0)
+    (property "Reference" "#PWR02401" (id 0) (at 146.05 76.2 0)
       (effects (font (size 1.27 1.27)) hide)
     )
@@
   (symbol (lib_id "power:+3V3") (at 165.1 173.99 0) (unit 1)
     (in_bom yes) (on_board yes) (fields_autoplaced)
-    (property "Reference" "#PWR0281" (id 0) (at 165.1 177.8 0)
+    (property "Reference" "#PWR02405" (id 0) (at 165.1 177.8 0)
       (effects (font (size 1.27 1.27)) hide)
     )
@@
   (symbol (lib_id "Device:R") (at 114.3 91.44 0) (unit 1)
     (in_bom yes) (on_board yes) (fields_autoplaced)
-    (property "Reference" "R101" (id 0) (at 116.84 90.1699 0)
+    (property "Reference" "R2401" (id 0) (at 116.84 90.1699 0)
       (effects (font (size 1.27 1.27)) (justify left))
     )
@@
   (symbol (lib_id "power:GND") (at 165.1 186.69 0) (unit 1)
     (in_bom yes) (on_board yes)
-    (property "Reference" "#PWR0282" (id 0) (at 165.1 193.04 0)
+    (property "Reference" "#PWR02406" (id 0) (at 165.1 193.04 0)
       (effects (font (size 1.27 1.27)) hide)
     )
