File: Power.kicad_sch (KiCad schematic)
At the start: 38 parts, among them J16 Screw_Terminal_01x02, J17 Screw_Terminal_01x02, J18 USB_C_Receptacle_USB2.0, Q3 Q_PMOS_GSD, U10 MCP45HV31-ST, U11 MCP45HV31-ST, U8 XL6009, U9 XL6009

Commit message: layout
Parts:
- removed C13: C, Capacitor_SMD:C_0805_2012Metric, symbol Device:C
- removed C14: C_Polarized, Capacitor_SMD:CP_Elec_8x10, symbol Device:C_Polarized
- removed C18: 47u, Capacitor_SMD:CP_Elec_8x10, symbol Device:C_Polarized
- removed C19: 1u, Capacitor_SMD:C_0805_2012Metric, symbol Device:C
- removed C20, C21, C22: 100n, Capacitor_SMD:C_0603_1608Metric, symbol Device:C
- removed D3, D4: D_Schottky, Diode_SMD:D_SMA-SMB_Universal_Handsoldering, symbol Device:D_Schottky
- removed F1: Polyfuse, Fuse:Fuse_1812_4532Metric, symbol Device:Polyfuse
- removed J16, J17: Screw_Terminal_01x02, TerminalBlock:TerminalBlock_bornier-2_P5.08mm, symbol Connector:Screw_Terminal_01x02
- removed J18: USB_C_Receptacle_USB2.0, Connector_USB:USB_C_Receptacle_HRO_TYPE-C-31-M-12, symbol Connector:USB_C_Receptacle_USB2.0
- removed L2: L, Inductor_SMD:L_12x12mm_H8mm, symbol Device:L
- removed Q3: Q_PMOS_GSD, Package_TO_SOT_SMD:SOT-23, symbol Device:Q_PMOS_GSD
- removed R15, R19, R20, R21: R, Resistor_SMD:R_0603_1608Metric, symbol Device:R
- removed R22: 100k, Resistor_SMD:R_0603_1608Metric, symbol Device:R
- removed TP4: TestPoint, TestPoint:TestPoint_Pad_D1.0mm, symbol Connector:TestPoint
- removed U11: MCP45HV31-ST, Package_SO:TSSOP-14_4.4x5mm_P0.65mm, symbol Potentiometer_Digital:MCP45HV31-ST
- removed U9: XL6009, Package_TO_SOT_SMD:TO-263-5_TabPin3, symbol XL6009:XL6009
- added C503: 100n, Capacitor_SMD:C_0603_1608Metric, symbol Device:C
- C501: renamed from C11; value C -> 1u
- C502: renamed from C12; value C_Polarized -> 220u
- L501: renamed from L1; value L -> 33uH
- R501: renamed from R14; value R -> 10k
- R502: renamed from R16; value R -> 10k
- R503: renamed from R17; value R -> 10k
- R504: renamed from R18; value R -> 470R
- TP501: renamed from TP3; value TestPoint -> Boost
- renumbered C15 to C504, C16 to C505, C17 to C506, C23 to C507, D2 to D501, U8 to U501, U10 to U502
Connections:
- net GND: now also C503.2
- net SW: now reaches D501.2 (A), L501.2, U501.3 (SW)
- net EN1 renamed EN
- net FB1 renamed FB
- net OUT1 renamed OUT
- net OUT: now also C503.1
- no-connect marks 10 -> 1
Other:
- note added: "OUT=1.25*(1+MCP/Rn) =1.25*(1+10k/470R)=27.8V"
- moved on the sheet: C501, C502, C504, C505, C506, D501, L501, R501, R502, R503, R504, TP501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
