File: RS232.kicad_sch (KiCad schematic)
At the start: 8 parts, among them J20 RS232_1, J21 RS232_2, U15 MAX3232

Commit message: layout
Parts:
- removed J20: RS232_1, Connector_PinHeader_2.54mm:PinHeader_1x03_P2.54mm_Vertical, symbol Connector:Conn_01x03_Female
- removed J21: RS232_2, Connector_PinHeader_2.54mm:PinHeader_1x03_P2.54mm_Vertical, symbol Connector:Conn_01x03_Female
- renumbered C29 to C801, C30 to C802, C31 to C803, C32 to C804, C33 to C805, U15 to U801
Connections:
- net RX1: now reaches U801.13 (R1IN)
- net TX1: now reaches U801.14 (T1OUT)
- net TX2: now reaches U801.7 (T2OUT)
- net RX2: now reaches U801.8 (R2IN)
Changed lines of the file:
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@@
 (kicad_sch (version 20211123) (generator eeschema)
   (paper "A4")
-  (wire (pts (xy 166.37 105.41) (xy 168.91 105.41))
+  (wire (pts (xy 166.37 115.57) (xy 170.18 115.57))
     (stroke (width 0) (type default) (color 0 0 0 0))
   )
@@
     (stroke (width 0) (type default) (color 0 0 0 0))
   )
-  (wire (pts (xy 166.37 115.57) (xy 180.34 115.57))
+  (wire (pts (xy 166.37 110.49) (xy 170.18 110.49))
     (stroke (width 0) (type default) (color 0 0 0 0))
   )
@@
     (stroke (width 0) (type default) (color 0 0 0 0))
   )
-  (wire (pts (xy 168.91 113.03) (xy 180.34 113.03))
-    (stroke (width 0) (type default) (color 0 0 0 0))
-  )
   (wire (pts (xy 176.53 95.25) (xy 177.8 95.25))
     (stroke (width 0) (type default) (color 0 0 0 0))
@@
     (stroke (width 0) (type default) (color 0 0 0 0))
   )
-  (wire (pts (xy 168.91 105.41) (xy 168.91 113.03))
-    (stroke (width 0) (type default) (color 0 0 0 0))
-  )
   (wire (pts (xy 146.05 129.54) (xy 146.05 128.27))
     (stroke (width 0) (type default) (color 0 0 0 0))
@@
     (stroke (width 0) (type default) (color 0 0 0 0))
   )
-  (wire (pts (xy 177.8 106.68) (xy 177.8 105.41))
-    (stroke (width 0) (type default) (color 0 0 0 0))
-  )
   (wire (pts (xy 125.73 100.33) (xy 121.92 100.33))
     (stroke (width 0) (type default) (color 0 0 0 0))
@@
     (stroke (width 0) (type default) (color 0 0 0 0))
   )
+  (wire (pts (xy 166.37 100.33) (xy 170.18 100.33))
+    (stroke (width 0) (type default) (color 0 0 0 0))
+  )
   (wire (pts (xy 166.37 87.63) (xy 168.91 87.63))
     (stroke (width 0) (type default) (color 0 0 0 0))
   )
-  (wire (pts (xy 177.8 105.41) (xy 180.34 105.41))
-    (stroke (width 0) (type default) (color 0 0 0 0))
-  )
-  (wire (pts (xy 177.8 118.11) (xy 177.8 119.38))
-    (stroke (width 0) (type default) (color 0 0 0 0))
-  )
   (wire (pts (xy 177.8 82.55) (xy 177.8 74.93))
     (stroke (width 0) (type default) (color 0 0 0 0))
   )
-  (wire (pts (xy 180.34 118.11) (xy 177.8 118.11))
-    (stroke (width 0) (type default) (color 0 0 0 0))
-  )
-  (wire (pts (xy 166.37 100.33) (xy 180.34 100.33))
-    (stroke (width 0) (type default) (color 0 0 0 0))
-  )
   (wire (pts (xy 146.05 67.31) (xy 146.05 66.04))
     (stroke (width 0) (type default) (color 0 0 0 0))
   )
-  (wire (pts (xy 166.37 110.49) (xy 171.45 110.49))
-    (stroke (width 0) (type default) (color 0 0 0 0))
-  )
   (wire (pts (xy 177.8 74.93) (xy 176.53 74.93))
     (stroke (width 0) (type default) (color 0 0 0 0))
@@
     (stroke (width 0) (type default) (color 0 0 0 0))
   )
-  (wire (pts (xy 171.45 102.87) (xy 180.34 102.87))
-    (stroke (width 0) (type default) (color 0 0 0 0))
-  )
   (wire (pts (xy 114.3 82.55) (xy 125.73 82.55))
     (stroke (width 0) (type default) (color 0 0 0 0))
   )
-  (wire (pts (xy 171.45 110.49) (xy 171.45 102.87))
-    (stroke (width 0) (type default) (color 0 0 0 0))
-  )
   (wire (pts (xy 166.37 82.55) (xy 177.8 82.55))
     (stroke (width 0) (type default) (color 0 0 0 0))
   )
+  (wire (pts (xy 166.37 105.41) (xy 170.18 105.41))
+    (stroke (width 0) (type default) (color 0 0 0 0))
+  )
+  (hierarchical_label "RX1" (shape input) (at 170.18 110.49 0)
+    (effects (font (size 1.27 1.27)) (justify left))
+  )
   (hierarchical_label "UART1_TX" (shape input) (at 121.92 100.33 180)
     (effects (font (size 1.27 1.27)) (justify right))
@@
     (effects (font (size 1.27 1.27)) (justify right))
   )
+  (hierarchical_label "TX2" (shape output) (at 170.18 105.41 0)
+    (effects (font (size 1.27 1.27)) (justify left))
+  )
+  (hierarchical_label "RX2" (shape input) (at 170.18 115.57 0)
+    (effects (font (size 1.27 1.27)) (justify left))
+  )
+  (hierarchical_label "TX1" (shape output) (at 170.18 100.33 0)
+    (effects (font (size 1.27 1.27)) (justify left))
+  )
   (symbol (lib_id "Interface_UART:MAX3232") (at 146.05 97.79 0) (unit 1)
     (in_bom yes) (on_board yes)
-    (property "Reference" "U15" (id 0) (at 146.05 53.34 0))
+    (property "Reference" "U801" (id 0) (at 146.05 53.34 0))
     (property "Value" "MAX3232" (id 1) (at 146.05 55.88 0))
     (property "Footprint" "Package_SO:SOIC-16_3.9x9.9mm_P1.27mm" (id 2) (at 147.32 124.46 0)
@@
   (symbol (lib_id "Device:C") (at 119.38 74.93 90) (unit 1)
     (in_bom yes) (on_board yes)
-    (property "Reference" "C29" (id 0) (at 120.65 68.58 90)
+    (property "Reference" "C801" (id 0) (at 120.65 68.58 90)
       (effects (font (size 1.27 1.27)) (justify left))
     )
@@
   (symbol (lib_id "Device:C") (at 172.72 74.93 270) (unit 1)
     (in_bom yes) (on_board yes)
-    (property "Reference" "C30" (id 0) (at 172.72 68.5292 90))
+    (property "Reference" "C802" (id 0) (at 172.72 68.5292 90))
     (property "Value" "100n" (id 1) (at 172.72 70.8406 90))
     (property "Footprint" "Capacitor_SMD:C_0603_1608Metric" (id 2) (at 168.91 75.8952 0)
@@
   (symbol (lib_id "power:+3V3") (at 146.05 66.04 0) (unit 1)
     (in_bom yes) (on_board yes)
-    (property "Reference" "#PWR0128" (id 0) (at 146.05 69.85 0)
+    (property "Reference" "#PWR0801" (id 0) (at 146.05 69.85 0)
       (effects (font (size 1.27 1.27)) hide)
     )
@@
   (symbol (lib_id "power:GND") (at 146.05 129.54 0) (unit 1)
     (in_bom yes) (on_board yes)
-    (property "Reference" "#PWR0133" (id 0) (at 146.05 135.89 0)
+    (property "Reference" "#PWR0806" (id 0) (at 146.05 135.89 0)
       (effects (font (size 1.27 1.27)) hide)
     )
@@
   (symbol (lib_id "Device:C") (at 172.72 95.25 270) (unit 1)
     (in_bom yes) (on_board yes)
-    (property "Reference" "C32" (id 0) (at 175.26 93.98 90))
+    (property "Reference" "C804" (id 0) (at 175.26 93.98 90))
     (property "Value" "100n" (id 1) (at 168.91 93.98 90))
     (property "Footprint" "Capacitor_SMD:C_0603_1608Metric" (id 2) (at 168.91 96.2152 0)
@@
   (symbol (lib_id "Device:C") (at 172.72 87.63 270) (unit 1)
     (in_bom yes) (on_board yes)
-    (property "Reference" "C31" (id 0) (at 175.26 86.36 90))
+    (property "Reference" "C803" (id 0) (at 175.26 86.36 90))
     (property "Value" "100n" (id 1) (at 168.91 86.36 90))
     (property "Footprint" "Capacitor_SMD:C_0603_1608Metric" (id 2) (at 168.91 88.5952 0)
@@
   (symbol (lib_id "power:GND") (at 177.8 95.25 90) (unit 1)
     (in_bom yes) (on_board yes)
-    (property "Reference" "#PWR0130" (id 0) (at 184.15 95.25 0)
+    (property "Reference" "#PWR0803" (id 0) (at 184.15 95.25 0)
       (effects (font (size 1.27 1.27)) hide)
     )
@@
   (symbol (lib_id "Device:C") (at 163.83 180.34 0) (unit 1)
     (in_bom yes) (on_board yes)
-    (property "Reference" "C33" (id 0) (at 166.751 179.1716 0)
+    (property "Reference" "C805" (id 0) (at 166.751 179.1716 0)
       (effects (font (size 1.27 1.27)) (justify left))
     )
@@
   (symbol (lib_id "power:GND") (at 163.83 185.42 0) (unit 1)
     (in_bom yes) (on_board yes)
-    (property "Reference" "#PWR0135" (id 0) (at 163.83 191.77 0)
+    (property "Reference" "#PWR0808" (id 0) (at 163.83 191.77 0)
       (effects (font (size 1.27 1.27)) hide)
     )
@@
   (symbol (lib_id "power:+3V3") (at 163.83 175.26 0) (unit 1)
     (in_bom yes) (on_board yes)
-    (property "Reference" "#PWR0134" (id 0) (at 163.83 179.07 0)
+    (property "Reference" "#PWR0807" (id 0) (at 163.83 179.07 0)
       (effects (font (size 1.27 1.27)) hide)
     )
@@
   (symbol (lib_id "power:+3V3") (at 177.8 87.63 270) (unit 1)
     (in_bom yes) (on_board yes)
-    (property "Reference" "#PWR0129" (id 0) (at 173.99 87.63 0)
+    (property "Reference" "#PWR0802" (id 0) (at 173.99 87.63 0)
       (effects (font (size 1.27 1.27)) hide)
     )
@@
     (pin "1")
   )
-  (symbol (lib_id "power:GND") (at 177.8 119.38 0) (unit 1)
-    (in_bom yes) (on_board yes)
-    (property "Reference" "#PWR0132" (id 0) (at 177.8 125.73 0)
-      (effects (font (size 1.27 1.27)) hide)
-    )
-    (property "Value" "GND" (id 1) (at 177.927 123.7742 0))
-    (property "Footprint" "" (id 2) (at 177.8 119.38 0)
-      (effects (font (size 1.27 1.27)) hide)
-    )
-    (property "Datasheet" "" (id 3) (at 177.8 119.38 0)
-      (effects (font (size 1.27 1.27)) hide)
-    )
-    (pin "1")
-  )
-  (symbol (lib_id "Connector:Conn_01x03_Female") (at 185.42 102.87 0) (unit 1)
-    (in_bom yes) (on_board yes)
-    (property "Reference" "J20" (id 0) (at 186.69 101.6 0)
-      (effects (font (size 1.27 1.27)) (justify left))
-    )
-    (property "Value" "RS232_1" (id 1) (at 186.69 104.14 0)
-      (effects (font (size 1.27 1.27)) (justify left))
-    )
-    (property "Footprint" "Connector_PinHeader_2.54mm:PinHeader_1x03_P2.54mm_Vertical" (id 2) (at 185.42 102.87 0)
-      (effects (font (size 1.27 1.27)) hide)
-    )
-    (property "Datasheet" "~" (id 3) (at 185.42 102.87 0)
-      (effects (font (size 1.27 1.27)) hide)
-    )
-    (pin "1")
-    (pin "2")
-    (pin "3")
-  )
-  (symbol (lib_id "power:GND") (at 177.8 106.68 0) (unit 1)
-    (in_bom yes) (on_board yes)
-    (property "Reference" "#PWR0131" (id 0) (at 177.8 113.03 0)
-      (effects (font (size 1.27 1.27)) hide)
-    )
-    (property "Value" "GND" (id 1) (at 177.927 111.0742 0))
-    (property "Footprint" "" (id 2) (at 177.8 106.68 0)
-      (effects (font (size 1.27 1.27)) hide)
-    )
-    (property "Datasheet" "" (id 3) (at 177.8 106.68 0)
-      (effects (font (size 1.27 1.27)) hide)
-    )
-    (pin "1")
-  )
-  (symbol (lib_id "Connector:Conn_01x03_Female") (at 185.42 115.57 0) (unit 1)
-    (in_bom yes) (on_board yes)
-    (property "Reference" "J21" (id 0) (at 186.69 114.3 0)
-      (effects (font (size 1.27 1.27)) (justify left))
-    )
-    (property "Value" "RS232_2" (id 1) (at 186.69 116.84 0)
-      (effects (font (size 1.27 1.27)) (justify left))
-    )
-    (property "Footprint" "Connector_PinHeader_2.54mm:PinHeader_1x03_P2.54mm_Vertical" (id 2) (at 185.42 115.57 0)
-      (effects (font (size 1.27 1.27)) hide)
-    )
-    (property "Datasheet" "~" (id 3) (at 185.42 115.57 0)
-      (effects (font (size 1.27 1.27)) hide)
-    )
-    (pin "1")
-    (pin "2")
-    (pin "3")
-  )
 )
