File: Relais.kicad_sch (KiCad schematic)
At the start: 24 parts, among them Q20 Q_NMOS_GSD, Q21 Q_NMOS_GSD, Q22 Q_NMOS_GSD, Q23 Q_NMOS_GSD

Commit message: layout
Parts:
- removed C62, C63, C64: 100n, Capacitor_SMD:C_0603_1608Metric, symbol Device:C
- removed D13, D14, D15, D16: D_Schottky, Diode_SMD:D_SMA-SMB_Universal_Handsoldering, symbol Device:D_Schottky
- removed Q21, Q22, Q23: Q_NMOS_GSD, Package_TO_SOT_SMD:SOT-23, symbol Device:Q_NMOS_GSD
- removed R85, R88, R89: 10k, Resistor_SMD:R_0603_1608Metric, symbol Device:R
- removed R87, R90, R91: 100k, Resistor_SMD:R_0603_1608Metric, symbol Device:R
- removed RLY1, RLY2, RLY3, RLY4: G5LE-14_DC5, Relay_THT:Relay_SPDT_Omron-G5LE-1, symbol dk_Power-Relays-Over-2-Amps:G5LE-14_DC5
- added D2501: 1N5819, Diode_SMD:D_SOD-323, symbol Diode:1N5819
- added K2501: G6K-2F-Y, Relay_SMD:Relay_DPDT_Omron_G6K-2F-Y, symbol Relay:AZ850-x
- renumbered C61 to C2001, Q20 to Q2001, R84 to R2001, R86 to R2003
Connections:
- net +5V: now also D2501.1 (K), K2501.1
- net COM1: now also K2501.3
- net COM2: now also K2501.6
- net NC1: now also K2501.2
- net NC2: now also K2501.7
- net NO1: now also K2501.4
- net NO2: now also K2501.5
- net at Q2001.3 (D): now also D2501.2 (A), K2501.8
- net IN1 renamed IN
Other:
- moved on the sheet: C2001, Q2001, R2001, R2003
