File: SD.kicad_sch (KiCad schematic)
At the start: 2 parts, among them J25 Micro_SD_Card_Det

Commit message: layout
Parts:
- removed J25: Micro_SD_Card_Det, symbol Connector:Micro_SD_Card_Det
- added U1601: TF-01A, SD:FT-01A, symbol sd:TF-01A
- renumbered C55 to C1601
Connections:
- net +3V3: now also U1601.4 (VDD)
- net CD: now also U1601.9 (CD)
- net CS: now also U1601.2 (CDDAT3(CS))
- net GND: now also U1601.10 (GND), U1601.11 (GND), U1601.12 (GND), U1601.13 (GND), U1601.6 (VSS)
- net MISO: now also U1601.7 (DAT0(D0))
- net MOSI: now also U1601.3 (CMD(DI))
- net SCK: now also U1601.5 (CLK(SCLK))
- no-connect marks 3 -> 2
Changed lines of the file:
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@@
 (kicad_sch (version 20211123) (generator eeschema)
   (paper "A4")
-  (no_connect (at 129.54 113.03))
-  (no_connect (at 129.54 90.17))
-  (no_connect (at 129.54 107.95))
+  (junction (at 144.78 118.11) (diameter 0) (color 0 0 0 0)
+  )
+  (junction (at 142.24 118.11) (diameter 0) (color 0 0 0 0)
+  )
+  (junction (at 139.7 118.11) (diameter 0) (color 0 0 0 0)
+  )
+  (no_connect (at 132.08 97.79))
+  (no_connect (at 132.08 95.25))
+  (wire (pts (xy 147.32 118.11) (xy 147.32 115.57))
+    (stroke (width 0) (type default) (color 0 0 0 0))
+  )
   (wire (pts (xy 166.37 176.53) (xy 166.37 179.07))
     (stroke (width 0) (type default) (color 0 0 0 0))
   )
-  (wire (pts (xy 124.46 92.71) (xy 129.54 92.71))
+  (wire (pts (xy 139.7 115.57) (xy 139.7 118.11))
     (stroke (width 0) (type default) (color 0 0 0 0))
   )
-  (wire (pts (xy 124.46 105.41) (xy 129.54 105.41))
+  (wire (pts (xy 139.7 118.11) (xy 142.24 118.11))
     (stroke (width 0) (type default) (color 0 0 0 0))
   )
@@
     (stroke (width 0) (type default) (color 0 0 0 0))
   )
-  (wire (pts (xy 173.99 120.65) (xy 173.99 113.03))
+  (wire (pts (xy 127 107.95) (xy 132.08 107.95))
     (stroke (width 0) (type default) (color 0 0 0 0))
   )
-  (wire (pts (xy 124.46 97.79) (xy 129.54 97.79))
+  (wire (pts (xy 144.78 118.11) (xy 144.78 115.57))
     (stroke (width 0) (type default) (color 0 0 0 0))
   )
-  (wire (pts (xy 124.46 100.33) (xy 129.54 100.33))
+  (wire (pts (xy 144.78 118.11) (xy 147.32 118.11))
     (stroke (width 0) (type default) (color 0 0 0 0))
   )
-  (wire (pts (xy 173.99 113.03) (xy 172.72 113.03))
+  (wire (pts (xy 157.48 95.25) (xy 157.48 97.79))
     (stroke (width 0) (type default) (color 0 0 0 0))
   )
-  (wire (pts (xy 124.46 110.49) (xy 129.54 110.49))
+  (wire (pts (xy 127 92.71) (xy 132.08 92.71))
     (stroke (width 0) (type default) (color 0 0 0 0))
   )
-  (wire (pts (xy 116.84 102.87) (xy 116.84 115.57))
+  (wire (pts (xy 142.24 118.11) (xy 144.78 118.11))
     (stroke (width 0) (type default) (color 0 0 0 0))
   )
-  (wire (pts (xy 124.46 95.25) (xy 129.54 95.25))
+  (wire (pts (xy 139.7 118.11) (xy 139.7 120.65))
     (stroke (width 0) (type default) (color 0 0 0 0))
   )
-  (wire (pts (xy 129.54 102.87) (xy 116.84 102.87))
+  (wire (pts (xy 142.24 118.11) (xy 142.24 115.57))
+    (stroke (width 0) (type default) (color 0 0 0 0))
+  )
+  (wire (pts (xy 154.94 95.25) (xy 157.48 95.25))
+    (stroke (width 0) (type default) (color 0 0 0 0))
+  )
+  (wire (pts (xy 127 102.87) (xy 132.08 102.87))
+    (stroke (width 0) (type default) (color 0 0 0 0))
+  )
+  (wire (pts (xy 160.02 92.71) (xy 154.94 92.71))
+    (stroke (width 0) (type default) (color 0 0 0 0))
+  )
+  (wire (pts (xy 127 105.41) (xy 132.08 105.41))
+    (stroke (width 0) (type default) (color 0 0 0 0))
+  )
+  (wire (pts (xy 127 100.33) (xy 132.08 100.33))
     (stroke (width 0) (type default) (color 0 0 0 0))
   )
@@
     (effects (font (size 1.27 1.27)) (justify left bottom))
   )
-  (hierarchical_label "MOSI" (shape input) (at 124.46 95.25 180)
+  (hierarchical_label "MISO" (shape output) (at 127 92.71 180)
     (effects (font (size 1.27 1.27)) (justify right))
   )
-  (hierarchical_label "MISO" (shape output) (at 124.46 105.41 180)
+  (hierarchical_label "SCK" (shape input) (at 127 105.41 180)
     (effects (font (size 1.27 1.27)) (justify right))
   )
-  (hierarchical_label "CD" (shape output) (at 124.46 110.49 180)
+  (hierarchical_label "MOSI" (shape input) (at 127 102.87 180)
     (effects (font (size 1.27 1.27)) (justify right))
   )
-  (hierarchical_label "SCK" (shape input) (at 124.46 100.33 180)
+  (hierarchical_label "CS" (shape input) (at 127 100.33 180)
     (effects (font (size 1.27 1.27)) (justify right))
   )
-  (hierarchical_label "CS" (shape input) (at 124.46 92.71 180)
+  (hierarchical_label "CD" (shape output) (at 127 107.95 180)
     (effects (font (size 1.27 1.27)) (justify right))
   )
-  (symbol (lib_id "Connector:Micro_SD_Card_Det") (at 152.4 100.33 0) (unit 1)
+  (symbol (lib_id "power:+3V3") (at 160.02 92.71 270) (unit 1)
     (in_bom yes) (on_board yes) (fields_autoplaced)
-    (property "Reference" "J25" (id 0) (at 153.035 78.74 0))
-    (property "Value" "Micro_SD_Card_Det" (id 1) (at 153.035 81.28 0))
-    (property "Footprint" "" (id 2) (at 204.47 82.55 0)
+    (property "Reference" "#PWR0137" (id 0) (at 156.21 92.71 0)
       (effects (font (size 1.27 1.27)) hide)
     )
-    (property "Datasheet" "https://www.hirose.com/product/en/download_file/key_name/DM3/category/Catalog/doc_file_id/49662/?file_category_id=4&item_id=195&is_series=1" (id 3) (at 152.4 97.79 0)
+    (property "Value" "+3V3" (id 1) (at 163.83 92.7101 90)
+      (effects (font (size 1.27 1.27)) (justify left))
+    )
+    (property "Footprint" "" (id 2) (at 160.02 92.71 0)
       (effects (font (size 1.27 1.27)) hide)
     )
-    (pin "1")
-    (pin "10")
-    (pin "11")
-    (pin "2")
-    (pin "3")
-    (pin "4")
-    (pin "5")
-    (pin "6")
-    (pin "7")
-    (pin "8")
-    (pin "9")
-  )
-  (symbol (lib_id "power:GND") (at 173.99 120.65 0) (unit 1)
-    (in_bom yes) (on_board yes) (fields_autoplaced)
-    (property "Reference" "#PWR0219" (id 0) (at 173.99 127 0)
-      (effects (font (size 1.27 1.27)) hide)
-    )
-    (property "Value" "GND" (id 1) (at 173.99 125.73 0))
-    (property "Footprint" "" (id 2) (at 173.99 120.65 0)
-      (effects (font (size 1.27 1.27)) hide)
-    )
-    (property "Datasheet" "" (id 3) (at 173.99 120.65 0)
+    (property "Datasheet" "" (id 3) (at 160.02 92.71 0)
       (effects (font (size 1.27 1.27)) hide)
     )
@@
   (symbol (lib_id "Device:C") (at 166.37 182.88 0) (unit 1)
     (in_bom yes) (on_board yes) (fields_autoplaced)
-    (property "Reference" "C55" (id 0) (at 170.18 181.6099 0)
+    (property "Reference" "C1601" (id 0) (at 170.18 181.6099 0)
       (effects (font (size 1.27 1.27)) (justify left))
     )
@@
   (symbol (lib_id "power:+3V3") (at 166.37 176.53 0) (unit 1)
     (in_bom yes) (on_board yes) (fields_autoplaced)
-    (property "Reference" "#PWR0220" (id 0) (at 166.37 180.34 0)
+    (property "Reference" "#PWR01604" (id 0) (at 166.37 180.34 0)
       (effects (font (size 1.27 1.27)) hide)
     )
@@
     (pin "1")
   )
-  (symbol (lib_id "power:GND") (at 116.84 115.57 0) (unit 1)
+  (symbol (lib_id "power:GND") (at 139.7 120.65 0) (unit 1)
     (in_bom yes) (on_board yes) (fields_autoplaced)
-    (property "Reference" "#PWR0218" (id 0) (at 116.84 121.92 0)
+    (property "Reference" "#PWR0136" (id 0) (at 139.7 127 0)
       (effects (font (size 1.27 1.27)) hide)
     )
-    (property "Value" "GND" (id 1) (at 116.84 120.65 0))
-    (property "Footprint" "" (id 2) (at 116.84 115.57 0)
+    (property "Value" "GND" (id 1) (at 139.7 125.73 0))
+    (property "Footprint" "" (id 2) (at 139.7 120.65 0)
       (effects (font (size 1.27 1.27)) hide)
     )
-    (property "Datasheet" "" (id 3) (at 116.84 115.57 0)
-      (effects (font (size 1.27 1.27)) hide)
-    )
-    (pin "1")
-  )
-  (symbol (lib_id "power:+3V3") (at 124.46 97.79 90) (unit 1)
-    (in_bom yes) (on_board yes) (fields_autoplaced)
-    (property "Reference" "#PWR0217" (id 0) (at 128.27 97.79 0)
-      (effects (font (size 1.27 1.27)) hide)
-    )
-    (property "Value" "+3V3" (id 1) (at 120.65 97.7899 90)
-      (effects (font (size 1.27 1.27)) (justify left))
-    )
-    (property "Footprint" "" (id 2) (at 124.46 97.79 0)
-      (effects (font (size 1.27 1.27)) hide)
-    )
-    (property "Datasheet" "" (id 3) (at 124.46 97.79 0)
+    (property "Datasheet" "" (id 3) (at 139.7 120.65 0)
       (effects (font (size 1.27 1.27)) hide)
     )
@@
   (symbol (lib_id "power:GND") (at 166.37 189.23 0) (unit 1)
     (in_bom yes) (on_board yes) (fields_autoplaced)
-    (property "Reference" "#PWR0221" (id 0) (at 166.37 195.58 0)
+    (property "Reference" "#PWR01605" (id 0) (at 166.37 195.58 0)
       (effects (font (size 1.27 1.27)) hide)
     )
@@
     (pin "1")
   )
+  (symbol (lib_id "power:GND") (at 157.48 97.79 0) (unit 1)
+    (in_bom yes) (on_board yes) (fields_autoplaced)
+    (property "Reference" "#PWR0138" (id 0) (at 157.48 104.14 0)
+      (effects (font (size 1.27 1.27)) hide)
+    )
+    (property "Value" "GND" (id 1) (at 157.48 102.87 0))
+    (property "Footprint" "" (id 2) (at 157.48 97.79 0)
+      (effects (font (size 1.27 1.27)) hide)
+    )
+    (property "Datasheet" "" (id 3) (at 157.48 97.79 0)
+      (effects (font (size 1.27 1.27)) hide)
+    )
+    (pin "1")
+  )
+  (symbol (lib_id "sd:TF-01A") (at 142.24 91.44 0) (unit 1)
+    (in_bom yes) (on_board yes) (fields_autoplaced)
+    (property "Reference" "U1601" (id 0) (at 143.51 85.09 0))
+    (property "Value" "TF-01A" (id 1) (at 143.51 87.63 0))
+    (property "Footprint" "SD:FT-01A" (id 2) (at 142.24 91.44 0)
+      (effects (font (size 1.27 1.27)) hide)
+    )
+    (property "Datasheet" "" (id 3) (at 142.24 91.44 0)
+      (effects (font (size 1.27 1.27)) hide)
+    )
+    (pin "1")
+    (pin "10")
+    (pin "11")
+    (pin "12")
+    (pin "13")
+    (pin "2")
+    (pin "3")
+    (pin "4")
+    (pin "5")
+    (pin "6")
+    (pin "7")
+    (pin "8")
+    (pin "9")
+  )
 )
