File: Shift.kicad_sch (KiCad schematic)
At the start: 6 parts, among them J26 DOUT_SHIFT, U21 TXB0104PW

Commit message: layout
Parts:
- R1701: renamed from R80; footprint Resistor_SMD:R_0201_0603Metric -> Resistor_SMD:R_0603_1608Metric
- renumbered C56 to C1701, C57 to C1702, J26 to J1701, JP14 to JP1701, U21 to U1701
Connections:
- net +3V3: now also JP1701.3 (B)
- net IN1: now also U1701.5 (A4); no longer U1701.2 (A1)
- net IN2: now also U1701.4 (A3); no longer U1701.3 (A2)
- net IN3: now also U1701.3 (A2); no longer U1701.4 (A3)
- net IN4: now also U1701.2 (A1); no longer U1701.5 (A4)
- net at J1701.1 (Pin_1): now also U1701.10 (B4); no longer U1701.13 (B1)
- net at J1701.2 (Pin_2): now also U1701.11 (B3); no longer U1701.12 (B2)
- net at J1701.3 (Pin_3): now also U1701.12 (B2); no longer U1701.11 (B3)
- net at J1701.4 (Pin_4): now also U1701.13 (B1); no longer U1701.10 (B4)
- no-connect marks 1 -> 0
Other:
- moved on the sheet: J1701
