File: Switch.kicad_sch (KiCad schematic)
At the start: 28 parts, among them Q10 MMBT3904, Q11 MMBT3904, Q4 Q_PMOS_GSD, Q5 Q_PMOS_GSD, Q6 MMBT3904, Q7 MMBT3904, Q8 Q_PMOS_GSD, Q9 Q_PMOS_GSD

Commit message: layout
Parts:
- removed C38, C39: 100n, Capacitor_SMD:C_0603_1608Metric, symbol Device:C
- C1002: renamed from C37; value 100n -> 1u; footprint Capacitor_SMD:C_0603_1608Metric -> Capacitor_SMD:C_0805_2012Metric
- renumbered C36 to C1001, Q4 to Q1001, Q5 to Q1002, Q6 to Q1003, Q7 to Q1004, Q8 to Q1005, Q9 to Q1006, Q10 to Q1007, Q11 to Q1008, R34 to R1001, R35 to R1002, R36 to R1003, R37 to R1004, R38 to R1005, R39 to R1006, R40 to R1007, R41 to R1008, R42 to R1009, R43 to R1010, R44 to R1011, R45 to R1012, R46 to R1013, R47 to R1014, R48 to R1015, R49 to R1016
Other:
- moved on the sheet: C1001, C1002
