File: embeddedBridge.kicad_pcb (KiCad board)
At the start: 2 copper layers, 293 parts, among them J1 AOUT, J10 IO2, J11 R1, J12 R2, J13 R3, J14 R4, J15 BAT, J16 Screw_Terminal_01x02, J17 Screw_Terminal_01x02, J18 USB_C_Receptacle_USB2.0, J19 CAN, J2 I2C1, J20 RS232_1, J21 RS232_2, J22 AIN, J23 CAN, J24 ESP8266, J26 DOUT_SHIFT, J3 I2C0, J4 Debug, J5 PWR, J6 DOUT1, J7 FOUT, J8 IO1, J9 DOUT2, Q1 Q_NPN_BCE, Q10 MMBT3904, Q11 MMBT3904, Q12 Q_PMOS_GSD, Q13 Q_PMOS_GSD, Q14 MMBT3904, Q15 MMBT3904, Q16 Q_PMOS_GSD, Q17 Q_PMOS_GSD, Q18 MMBT3904, Q19 MMBT3904, Q2 Q_PNP_BCE, Q20 Q_NMOS_GSD, Q21 Q_NMOS_GSD, Q22 Q_NMOS_GSD, Q23 Q_NMOS_GSD, Q3 Q_PMOS_GSD, Q4 Q_PMOS_GSD, Q5 Q_PMOS_GSD, Q6 MMBT3904, Q7 MMBT3904, Q8 Q_PMOS_GSD, Q9 Q_PMOS_GSD, SW1 RESET, U1 Pico, U10 MCP45HV31-ST, U11 MCP45HV31-ST, U12 TJA1051T-3, U13 MCP2515-xSO, U14 LM324, U15 MAX3232, U16 MCP4728, U17 ADS1115IDGS, U18 TJA1051T-3, U19 MCP2515-xSO, U2 INA219AxDCN, U20 AD9833xRM, U21 TXB0104PW, U22 24LC32, U23 INA219AxDCN, U24 INA219AxDCN, U26 Opamp_Dual, U27 MCP4725xxx-xCH, U28 MCP23017_SS, U3 ISO1540, U4 MCP4725xxx-xCH, U5 Opamp_Dual, U6 INA219AxDCN, U7 INA219AxDCN, U8 XL6009, U9 XL6009, X1 XO32, Y1 Crystal, Y2 Crystal

Commit message: layout
Parts:
- removed C13: C, Capacitor_SMD:C_0805_2012Metric
- removed C14: C_Polarized, Capacitor_SMD:CP_Elec_8x10
- removed C18: 47u, Capacitor_SMD:CP_Elec_8x10
- removed C19: 1u, Capacitor_SMD:C_0805_2012Metric
- removed C20, C21, C22, C37, C38, C41, C42, C52, C60, C61, C62, C71, C72: 100n, Capacitor_SMD:C_0603_1608Metric
- removed C34: 10u, Capacitor_SMD:C_0805_2012Metric
- removed D1, D11, D13, D14, D15, D16, D3, D4, D5, D6, D7, D9: D_Schottky, Diode_SMD:D_SMA-SMB_Universal_Handsoldering
- removed D10, D12, D8: D_Zener, Diode_SMD:D_SMA-SMB_Universal_Handsoldering
- removed F1: Polyfuse, Fuse:Fuse_1812_4532Metric
- removed J10: IO2, Connector_PinHeader_2.54mm:PinHeader_1x03_P2.54mm_Vertical
- removed J11: R1, Connector_PinHeader_2.54mm:PinHeader_1x03_P2.54mm_Vertical
- removed J12: R2, Connector_PinHeader_2.54mm:PinHeader_1x03_P2.54mm_Vertical
- removed J13: R3, Connector_PinHeader_2.54mm:PinHeader_1x03_P2.54mm_Vertical
- removed J14: R4, Connector_PinHeader_2.54mm:PinHeader_1x03_P2.54mm_Vertical
- removed J16, J17: Screw_Terminal_01x02, TerminalBlock:TerminalBlock_bornier-2_P5.08mm
- removed J18: USB_C_Receptacle_USB2.0, Connector_USB:USB_C_Receptacle_HRO_TYPE-C-31-M-12
- removed J19, J23: CAN, Connector_PinHeader_2.54mm:PinHeader_1x03_P2.54mm_Vertical
- removed J20: RS232_1, Connector_PinHeader_2.54mm:PinHeader_1x03_P2.54mm_Vertical
- removed J21: RS232_2, Connector_PinHeader_2.54mm:PinHeader_1x03_P2.54mm_Vertical
- removed J5: PWR, Connector_PinHeader_2.54mm:PinHeader_1x05_P2.54mm_Vertical
- removed J8: IO1, Connector_PinHeader_2.54mm:PinHeader_1x03_P2.54mm_Vertical
- removed J9: DOUT2, Connector_PinHeader_2.54mm:PinHeader_1x05_P2.54mm_Vertical
- removed JP10: A2, Jumper:SolderJumper-2_P1.3mm_Open_Pad1.0x1.5mm
- removed JP11: A3, Jumper:SolderJumper-2_P1.3mm_Open_Pad1.0x1.5mm
- removed JP13, JP7: CAN_term, Connector_PinHeader_2.54mm:PinHeader_1x03_P2.54mm_Vertical
- removed JP2: DOUT1, Jumper:SolderJumper-2_P1.3mm_Bridged_Pad1.0x1.5mm
- removed JP3: DOUT2, Jumper:SolderJumper-2_P1.3mm_Bridged_Pad1.0x1.5mm
- removed JP4: DOUT3, Jumper:SolderJumper-2_P1.3mm_Bridged_Pad1.0x1.5mm
- removed JP5: DOUT4, Jumper:SolderJumper-2_P1.3mm_Bridged_Pad1.0x1.5mm
- removed JP9: A1, Jumper:SolderJumper-2_P1.3mm_Open_Pad1.0x1.5mm
- removed L2: L, Inductor_SMD:L_12x12mm_H8mm
- removed Q21, Q22, Q23: Q_NMOS_GSD, Package_TO_SOT_SMD:SOT-23
- removed Q3: Q_PMOS_GSD, Package_TO_SOT_SMD:SOT-23
- removed the R101 at (280.0, 73.7)
- removed R15, R19, R20, R21: R, Resistor_SMD:R_0603_1608Metric
- removed R22, R87, R90, R91: 100k, Resistor_SMD:R_0603_1608Metric
- removed R85, R88, R89: 10k, Resistor_SMD:R_0603_1608Metric
- removed RLY1, RLY2, RLY3, RLY4: G5LE-14_DC5, Relay_THT:Relay_SPDT_Omron-G5LE-1
- removed TP4: TestPoint, TestPoint:TestPoint_Pad_D1.0mm
- removed U11: MCP45HV31-ST, Package_SO:TSSOP-14_4.4x5mm_P0.65mm
- removed U9: XL6009, Package_TO_SOT_SMD:TO-263-5_TabPin3
- added C1501: 100n, Capacitor_SMD:C_0603_1608Metric, F.Cu at (8.00, 29.7)
- added C2101: 1u, Capacitor_SMD:C_0805_2012Metric, F.Cu at (91.0, 38.1)
- added C2102: 220u, Capacitor_SMD:CP_Elec_8x10, F.Cu at (89.2, 43.9)
- added C2103: 100n, Capacitor_SMD:C_0603_1608Metric, F.Cu at (81.0, 40.5)
- added C2104: 47u, Capacitor_SMD:CP_Elec_8x10, F.Cu at (82.6, 4.57)
- added C2105: 1u, Capacitor_SMD:C_0805_2012Metric, F.Cu at (90.0, 6.60)
- added C2106: 100n, Capacitor_SMD:C_0603_1608Metric, F.Cu at (90.2, 8.38)
- added C2107: 100n, Capacitor_SMD:C_0603_1608Metric, B.Cu at (94.6, 40.4)
- added C2501: 100n, Capacitor_SMD:C_0603_1608Metric, F.Cu at (44.3, 11.7)
- added C2601: 100n, Capacitor_SMD:C_0603_1608Metric, B.Cu at (79.0, 73.7)
- added C503: 100n, Capacitor_SMD:C_0603_1608Metric, F.Cu at (60.6, 40.5)
- added C508: 100n, Capacitor_SMD:C_0603_1608Metric, B.Cu at (91.5, 58.5)
- added C509: 100n, Capacitor_SMD:C_0603_1608Metric, F.Cu at (82.8, 55.6)
- added C901: 100n, Capacitor_SMD:C_0603_1608Metric, B.Cu at (80.5, 92.5)
- added D101: 1N5819, Diode_SMD:D_SOD-323, F.Cu at (41.7, 4.32)
- added D201: 1N5819, Diode_SMD:D_SOD-323, F.Cu at (46.2, 15.1)
- added D2101: D_Schottky, Diode_SMD:D_SMA-SMB_Universal_Handsoldering, F.Cu at (82.9, 37.1)
- added D2102: 1N5819, Diode_SMD:D_SOD-323, F.Cu at (45.6, 91.5)
- added D2103: 1N5819, Diode_SMD:D_SOD-323, B.Cu at (45.6, 91.5)
- added D2104: 1N5819, Diode_SMD:D_SOD-323, F.Cu at (48.2, 91.5)
- added D2105: 1N5819, Diode_SMD:D_SOD-323, B.Cu at (48.2, 91.5)
- added D2106: 1N5819, Diode_SMD:D_SOD-323, F.Cu at (50.7, 91.5)
- added D2107: 1N5819, Diode_SMD:D_SOD-323, B.Cu at (50.7, 91.5)
- added D2108: 1N5819, Diode_SMD:D_SOD-323, F.Cu at (53.3, 91.5)
- added D2109: 1N5819, Diode_SMD:D_SOD-323, B.Cu at (53.3, 91.5)
- added D2501: 1N5819, Diode_SMD:D_SOD-323, F.Cu at (80.9, 80.4)
- added D2601: 1N5819, Diode_SMD:D_SOD-323, B.Cu at (80.9, 73.5)
- added F2501: Polyfuse, Fuse:Fuse_1812_4532Metric, F.Cu at (48.3, 11.3)
- added H101: MountingHole_Pad, MountingHole:MountingHole_3.2mm_M3_DIN965_Pad, F.Cu at (5.00, 5.00)
- added H102: MountingHole_Pad, MountingHole:MountingHole_3.2mm_M3_DIN965_Pad, F.Cu at (95.0, 5.00)
- added H103: MountingHole_Pad, MountingHole:MountingHole_3.2mm_M3_DIN965_Pad, F.Cu at (5.00, 95.0)
- added H104: MountingHole_Pad, MountingHole:MountingHole_3.2mm_M3_DIN965_Pad, F.Cu at (95.0, 95.0)
- added J105: VCC, Connector_PinHeader_2.54mm:PinHeader_1x02_P2.54mm_Vertical, F.Cu at (58.7, 50.9)
- added J108: CAN1, Connector_PinHeader_2.54mm:PinHeader_1x03_P2.54mm_Vertical, F.Cu at (1.91, 54.8)
- added J109: CAN2, Connector_PinHeader_2.54mm:PinHeader_1x03_P2.54mm_Vertical, F.Cu at (1.78, 66.9)
- added J110: VDC, Connector_PinHeader_2.54mm:PinHeader_1x02_P2.54mm_Vertical, F.Cu at (79.1, 50.9)
- added J111: R1_1, Connector_PinHeader_2.54mm:PinHeader_1x03_P2.54mm_Vertical, F.Cu at (94.6, 80.0)
- added J112: R1_2, Connector_PinHeader_2.54mm:PinHeader_1x03_P2.54mm_Vertical, F.Cu at (94.6, 71.3)
- added J113: R2_1, Connector_PinHeader_2.54mm:PinHeader_1x03_P2.54mm_Vertical, F.Cu at (98.3, 71.3)
- added J114: R2_2, Connector_PinHeader_2.54mm:PinHeader_1x03_P2.54mm_Vertical, F.Cu at (98.3, 80.0)
- added J115: RS232_2, Connector_PinHeader_2.54mm:PinHeader_1x03_P2.54mm_Vertical, F.Cu at (1.91, 18.8)
- added J116: RS232_1, Connector_PinHeader_2.54mm:PinHeader_1x03_P2.54mm_Vertical, F.Cu at (1.91, 10.0)
- added J117: +3V3, Connector_PinHeader_2.54mm:PinHeader_1x02_P2.54mm_Vertical, F.Cu at (50.2, 31.4)
- added J118: +5V, Connector_PinHeader_2.54mm:PinHeader_1x02_P2.54mm_Vertical, F.Cu at (50.2, 27.7)
- added J2501: USB_C_Receptacle_USB2.0, Connector_USB:USB_C_Receptacle_HRO_TYPE-C-31-M-12, F.Cu at (48.3, 3.81)
- added K2501: G6K-2F-Y, Relay_SMD:Relay_DPDT_Omron_G6K-2F-Y, F.Cu at (87.4, 76.8)
- added K2601: G6K-2F-Y, Relay_SMD:Relay_DPDT_Omron_G6K-2F-Y, B.Cu at (87.4, 76.8)
- added L2101: 33uH, Inductor_SMD:L_12x12mm_H8mm, F.Cu at (84.7, 16.0)
- added Q2501: Q_PMOS_GSD, Package_TO_SOT_SMD:SOT-23, F.Cu at (49.3, 15.1)
- added Q2601: Q_NMOS_GSD, Package_TO_SOT_SMD:SOT-23, B.Cu at (80.0, 77.0)
- added R2101: 10k, Resistor_SMD:R_0603_1608Metric, F.Cu at (95.6, 31.2)
- added R2102: 10k, Resistor_SMD:R_0603_1608Metric, B.Cu at (91.5, 40.4)
- added R2103: 10k, Resistor_SMD:R_0603_1608Metric, B.Cu at (89.5, 35.3)
- added R2104: 470R, Resistor_SMD:R_0603_1608Metric, B.Cu at (94.6, 30.7)
- added R2401: 10k, Resistor_SMD:R_0603_1608Metric, B.Cu at (58.7, 69.4)
- added R2501: 100k, Resistor_SMD:R_0603_1608Metric, F.Cu at (44.3, 15.1)
- added R2601: 10k, Resistor_SMD:R_0603_1608Metric, B.Cu at (79.0, 80.4)
- added R2602: 100k, Resistor_SMD:R_0603_1608Metric, B.Cu at (81.1, 80.3)
- added REF**: OSHW-Logo2_7.3x6mm_SilkScreen, Symbol:OSHW-Logo2_7.3x6mm_SilkScreen, F.Cu at (44.2, 65.3)
- added TP201: VBUS, TestPoint:TestPoint_Pad_D1.0mm, B.Cu at (48.6, 11.3)
- added TP202: +5V, TestPoint:TestPoint_Pad_D1.0mm, B.Cu at (54.2, 15.1)
- added TP2101: Boost, TestPoint:TestPoint_Pad_D1.0mm, B.Cu at (85.2, 42.9)
- added U1601: TF-01A, SD:FT-01A, B.Cu at (25.1, 92.0)
- added U2101: XL6009, Package_TO_SOT_SMD:TO-263-5_TabPin3, F.Cu at (86.2, 28.7)
- added U2102: MCP45HV31-ST, Package_SO:TSSOP-14_4.4x5mm_P0.65mm, B.Cu at (93.0, 35.6)
- added U2301: PDS1-M, PDS1:PSD1, F.Cu at (35.4, 88.3)
- C1002: renamed from C36; value 100n -> 1u; footprint Capacitor_SMD:C_0603_1608Metric -> Capacitor_SMD:C_0805_2012Metric
- C1101: renamed from C39; moved to B.Cu
- C1102: renamed from C40; value 100n -> 1u; footprint Capacitor_SMD:C_0603_1608Metric -> Capacitor_SMD:C_0805_2012Metric
- C1201: renamed from C43; moved to F.Cu
- C1301: renamed from C44; moved to B.Cu
- C1302: renamed from C45; value 100n -> 22p; moved to B.Cu
- C1303: renamed from C46; moved to B.Cu
- C1304: renamed from C47; value 22p -> 100n
- C1401: renamed from C48; moved to B.Cu
- C1402: renamed from C49; value 100n -> 10n; moved to B.Cu
- C1403: renamed from C50; value 10n -> 20p; moved to B.Cu
- C1404: renamed from C51; value 20p -> 100n; moved to B.Cu
- C1601: renamed from C53; moved to B.Cu
- C1801: renamed from C56; moved to B.Cu
- C1901: renamed from C57; moved to B.Cu
- C1902: renamed from C58; moved to B.Cu
- C201: renamed from C1; moved to B.Cu
- C203: renamed from C3; value 100n -> 1u; footprint Capacitor_SMD:C_0603_1608Metric -> Capacitor_SMD:C_0805_2012Metric
- C204: renamed from C4; value 100n -> 1u; footprint Capacitor_SMD:C_0603_1608Metric -> Capacitor_SMD:C_0805_2012Metric
- C205: renamed from C5; moved to B.Cu
- C2301: renamed from C65; moved to B.Cu
- C2302: renamed from C66; moved to B.Cu
- C2303: renamed from C67; value 100n -> 680n; moved to B.Cu
- C2304: renamed from C68; moved to B.Cu
- C2305: renamed from C69; value C -> 100n
- C2401: renamed from C70; moved to B.Cu
- C301: renamed from C7; moved to B.Cu
- C302: renamed from C8; moved to B.Cu
- C401: renamed from C9; moved to B.Cu
- C402: renamed from C10; moved to B.Cu
- C501: renamed from C11; value C -> 1u
- C502: renamed from C12; value C_Polarized -> 220u
- C507: renamed from C23; moved to B.Cu
- C601: renamed from C24; moved to B.Cu
- C602: renamed from C25; moved to B.Cu
- C603: renamed from C26; moved to B.Cu
- J102: renamed from J2; footprint Connector_JST:JST_PH_B2B-PH-K_1x02_P2.00mm_Vertical -> Connector_JST:JST_PH_B3B-PH-K_1x03_P2.00mm_Vertical
- JP101: renamed from JP1; moved to B.Cu
- JP2301: renamed from JP15; value Jumper_3_Open -> DDS AMP
- JP601: renamed from JP6; moved to B.Cu
- JP701: renamed from JP8; value Jumper_3_Open -> DAC AMP
- L501: renamed from L1; value L -> 33uH
- R101: renamed from R1; moved to B.Cu
- R102: renamed from R2; moved to B.Cu
- R1201: renamed from R66; value R -> 12k
- R1202: renamed from R67; value R -> 1k5; moved to B.Cu
- R1203: renamed from R68; value R -> 12k
- R1204: renamed from R69; value R -> 1k5; moved to B.Cu
- R1205: renamed from R70; value R -> 12k
- R1206: renamed from R71; value R -> 1k5; moved to B.Cu
- R1207: renamed from R72; value R -> 12k
- R1208: renamed from R73; value R -> 1k5; moved to B.Cu
- R1501: renamed from R76; footprint Resistor_SMD:R_0201_0603Metric -> Resistor_SMD:R_0603_1608Metric
- R1502: renamed from R77; footprint Resistor_SMD:R_0201_0603Metric -> Resistor_SMD:R_0603_1608Metric
- R1503: renamed from R78; footprint Resistor_SMD:R_0201_0603Metric -> Resistor_SMD:R_0603_1608Metric
- R1504: renamed from R79; footprint Resistor_SMD:R_0201_0603Metric -> Resistor_SMD:R_0603_1608Metric
- R1701: renamed from R80; footprint Resistor_SMD:R_0201_0603Metric -> Resistor_SMD:R_0603_1608Metric
- R1901: renamed from R81; moved to B.Cu
- R1903: renamed from R83; moved to B.Cu
- R201: renamed from R3; moved to B.Cu
- R202: renamed from R4; moved to B.Cu
- R203: renamed from R5; moved to B.Cu
- R204: renamed from R6; moved to B.Cu
- R2301: renamed from R95; value 5k -> 4k7; moved to B.Cu
- R2302: renamed from R96; value 40k -> 39k; moved to B.Cu
- R2303: renamed from R97; moved to B.Cu
- R2304: renamed from R98; moved to B.Cu
- R301: renamed from R8; moved to B.Cu
- R303: renamed from R10; moved to B.Cu
- R401: renamed from R11; moved to B.Cu
- R402: renamed from R12; moved to B.Cu
- R403: renamed from R13; moved to B.Cu
- R501: renamed from R14; value R -> 10k; moved to F.Cu
- R502: renamed from R16; value R -> 10k; moved to B.Cu
- R503: renamed from R17; value R -> 10k; moved to B.Cu
- R504: renamed from R18; value R -> 470R; moved to B.Cu
- R701: renamed from R25; value R -> 10k
- R702: renamed from R26; value R -> 10k
- R703: renamed from R27; value R -> 68k
- R704: renamed from R28; value R -> 68k
- R705: renamed from R29; value R -> 10k
- R706: renamed from R30; value R -> 10k
- R707: renamed from R31; value R -> 68k
- R708: renamed from R32; value R -> 68k
- R901: renamed from R33; moved to B.Cu
- TP101: renamed from TP1; value TestPoint -> +3V3; moved to B.Cu
- TP102: renamed from TP2; value TestPoint -> DDS; moved to B.Cu
- TP501: renamed from TP3; value TestPoint -> Boost; moved to B.Cu
- U1301: renamed from U18; moved to B.Cu
- U1401: renamed from U20; moved to B.Cu
- U1801: renamed from U22; moved to B.Cu
- U1901: renamed from U23; moved to B.Cu
- U201: renamed from U2; moved to B.Cu
- U203: renamed from U4; moved to B.Cu
- U2302: renamed from U26; moved to B.Cu
- U2303: renamed from U27; moved to B.Cu
- U2401: renamed from U28; moved to B.Cu
- U301: renamed from U6; moved to B.Cu
- U401: renamed from U7; moved to B.Cu
- U502: renamed from U10; moved to B.Cu
- U601: renamed from U12; moved to B.Cu
- U901: renamed from U16; moved to B.Cu
- X1401: renamed from X1; moved to B.Cu
- Y1301: renamed from Y2; value Crystal -> 8MHz; footprint Crystal:Crystal_SMD_HC49-SD -> Crystal:Crystal_SMD_5032-2Pin_5.0x3.2mm; moved to B.Cu
- Y601: renamed from Y1; value Crystal -> 8MHz; footprint Crystal:Crystal_SMD_HC49-SD -> Crystal:Crystal_SMD_5032-2Pin_5.0x3.2mm; moved to B.Cu
- moved C2305 313.6 mm to (28.2, 84.6), turned to 90 degrees
- moved R2304 312.1 mm to (41.3, 93.9)
- moved R2302 310.0 mm to (38.2, 91.6), turned to 180 degrees
- moved JP2301 309.1 mm to (34.8, 98.2), turned to -90 degrees
- moved R2303 305.9 mm to (38.2, 93.9), turned to 180 degrees
- moved U2303 302.6 mm to (41.5, 90.3), turned to 90 degrees
- moved C2304 302.3 mm to (42.5, 86.6), turned to 90 degrees
- moved R2301 302.1 mm to (38.2, 89.9), turned to 180 degrees
- moved U2302 301.9 mm to (32.8, 93.6), turned to 180 degrees
- moved C2303 290.5 mm to (41.3, 95.5)
- moved C2201 286.9 mm to (73.6, 87.8), turned to 0 degrees
- moved C2202 285.5 mm to (76.4, 85.2), turned to 90 degrees
- moved Q2001 281.5 mm to (80.0, 77.0), turned to 0 degrees
- moved C2301 278.8 mm to (28.2, 92.4), turned to -90 degrees
- moved R2003 275.2 mm to (81.1, 73.7), turned to 90 degrees
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- renumbered C35 to C1001, C54 to C1701, C55 to C1702, C59 to C2001, C2 to C202, C6 to C206, C63 to C2201, C64 to C2202, C15 to C504, C16 to C505, C17 to C506, C27 to C604, C28 to C701, C29 to C801, C30 to C802, C31 to C803, C32 to C804, C33 to C805, D2 to D501, J1 to J101, J3 to J103, J4 to J104, J6 to J106, J7 to J107, J22 to J1201, J24 to J1501, J26 to J1701, J15 to J201, JP12 to JP1301, JP14 to JP1701, PS1 to PS201, Q4 to Q1001, Q5 to Q1002, Q6 to Q1003, Q7 to Q1004, Q8 to Q1005, Q9 to Q1006, Q10 to Q1007, Q11 to Q1008, Q12 to Q1101, Q13 to Q1102, Q14 to Q1103, Q15 to Q1104, Q16 to Q1105, Q17 to Q1106, Q18 to Q1107, Q19 to Q1108, Q20 to Q2001, Q1 to Q201, Q2 to Q202, R34 to R1001, R35 to R1002, R36 to R1003, R37 to R1004, R38 to R1005, R39 to R1006, R40 to R1007, R41 to R1008, R42 to R1009, R43 to R1010, R44 to R1011, R45 to R1012, R46 to R1013, R47 to R1014, R48 to R1015, R49 to R1016, R50 to R1101, R51 to R1102, R52 to R1103, R53 to R1104, R54 to R1105, R55 to R1106, R56 to R1107, R57 to R1108, R58 to R1109, R59 to R1110, R60 to R1111, R61 to R1112, R62 to R1113, R63 to R1114, R64 to R1115, R65 to R1116, R74 to R1301, R75 to R1302, R82 to R1902, R84 to R2001, R86 to R2003, R7 to R205, R92 to R2201, R93 to R2202, R94 to R2203, R9 to R302, R23 to R601, R24 to R602, SW1 to SW101, U1 to U101, U17 to U1201, U19 to U1302, U21 to U1701, U3 to U202, U5 to U204, U24 to U2201, U8 to U501, U13 to U602, U14 to U701, U15 to U801
Connections:
- net /DOUT1_VCC renamed /IO_Expander/GPA1
- net /DOUT1_VDC renamed /IO_Expander/GPB1
- net /DOUT2_VCC renamed /IO_Expander/GPA2
- net /DOUT2_VDC renamed /IO_Expander/GPB2
- net /DOUT3_VCC renamed /IO_Expander/GPA3
- net /DOUT3_VDC renamed /IO_Expander/GPB3
- net /DOUT4_VCC renamed /IO_Expander/GPA4
- net /DOUT4_VDC renamed /IO_Expander/GPB4
- net /Power/FB1 renamed /Power1/FB
- net Net-(D2-Pad2) renamed /Power1/SW
- net Net-(Q1-Pad3) renamed /Battery/BAT+_
- C1001 pad 1: +3V3 -> VCC
- C1101 pad 1: VCC -> VDC
- C1201 pad 1: VDC -> +3V3
- C1301 pad 1: +3V3 -> Net-(C1301-Pad1)
- C1302 pad 1: Net-(C45-Pad1) -> Net-(C1302-Pad1)
- C1303 pad 1: Net-(C46-Pad1) -> Net-(C1303-Pad1)
- C1304 pad 1: Net-(C47-Pad1) -> +3V3
- C1401 pad 1: +3V3 -> Net-(C1401-Pad1)
- C1402 pad 1: Net-(C49-Pad1) -> +3V3
- C1402 pad 2: GND -> Net-(C1402-Pad2)
- C1403 pad 1: +3V3 -> /AMP_offset/IN
- C1403 pad 2: Net-(C50-Pad2) -> GND
- C1404 pad 1: /AMP_offset/IN -> +3V3
- C1701 pad 1: +3V3 -> Net-(C1701-Pad1)
- C1801 pad 1: Net-(C56-Pad1) -> +3V3
- C1901 pad 1: +3V3 -> Net-(C1901-Pad1)
- C1901 pad 2: GND -> Net-(C1901-Pad2)
- C2001 pad 1: Net-(C59-Pad1) -> +5V
- C2001 pad 2: Net-(C59-Pad2) -> GND
- C2201 pad 1: +5V -> Net-(C2201-Pad1)
- C2201 pad 2: GND -> Net-(C2201-Pad2)
- C2202 pad 1: +5V -> +3V3
- C2301 pad 1: Net-(C65-Pad1) -> Net-(C2301-Pad1)
- C2301 pad 2: Net-(C65-Pad2) -> Net-(C2301-Pad2)
- C2302 pad 1: +3V3 -> Net-(C2301-Pad2)
- C2302 pad 2: GND -> Net-(C2302-Pad2)
- C2303 pad 1: Net-(C67-Pad1) -> Net-(C2303-Pad1)
- C2303 pad 2: Net-(C67-Pad2) -> GND
- C2304 pad 1: Net-(C67-Pad2) -> +3V3
- C2304 pad 2: Net-(C68-Pad2) -> GND
- C2305 pad 1: Net-(C69-Pad1) -> +3V3
- J1701 pad 1: Net-(J26-Pad1) -> Net-(J1701-Pad1)
- J1701 pad 2: Net-(J26-Pad2) -> Net-(J1701-Pad2)
- J1701 pad 3: Net-(J26-Pad3) -> Net-(J1701-Pad3)
- J1701 pad 4: Net-(J26-Pad4) -> Net-(J1701-Pad4)
- JP1301 pad 2: Net-(C45-Pad1) -> Net-(C1301-Pad1)
- JP1701 pad 2: Net-(C56-Pad1) -> Net-(C1701-Pad1)
- JP1701 pad 3: unconnected-(JP14-Pad3) -> +3V3
- JP2301 pad 1: Net-(C68-Pad2) -> Net-(C2302-Pad2)
- JP2301 pad 3: Net-(C67-Pad2) -> Net-(C2301-Pad2)
- Q1101 pad 3: /Switch2/DOUT1 -> /Cu4+
- Q1102 pad 3: /Switch2/DOUT2 -> /Cu3+
- Q1105 pad 3: /Switch2/DOUT3 -> /Switch1/DOUT3
- Q1106 pad 3: /Switch2/DOUT4 -> /Switch1/DOUT4
- Q201 pad 1: Net-(Q1-Pad1) -> Net-(Q201-Pad1)
- Q202 pad 1: Net-(Q1-Pad1) -> Net-(Q201-Pad1)
- R1301 pad 1: Net-(J23-Pad1) -> /CAN1/CANL
- R1301 pad 2: Net-(JP13-Pad2) -> /CAN1/CANH
- R1901 pad 2: Net-(C59-Pad1) -> Net-(C1901-Pad1)
- R1903 pad 2: Net-(C59-Pad2) -> Net-(C1901-Pad2)
- R2001 pad 1: /R1 -> /Relais1
- R201 pad 2: Net-(R3-Pad2) -> /Battery/SDA_
- R202 pad 2: Net-(R4-Pad2) -> /Battery/SCL_
- R2201 pad 2: Net-(C65-Pad1) -> Net-(C2201-Pad1)
- R2203 pad 2: Net-(C65-Pad2) -> Net-(C2201-Pad2)
- R2303 pad 1: Net-(C69-Pad1) -> Net-(C2303-Pad1)
- R2304 pad 1: Net-(C69-Pad1) -> Net-(C2303-Pad1)
- R601 pad 1: Net-(J19-Pad1) -> /CAN2/CANL
- R601 pad 2: Net-(JP7-Pad2) -> /CAN2/CANH
- U101 pad 10: /R2 -> /SPI0_CS_SD
- U101 pad 19: /R3 -> /SPI0_CS_CAN2
- U101 pad 20: /R4 -> /SPI0_CS_CAN1
- U101 pad 22: /SPI0_CS_SD -> /CD_SD
- U101 pad 26: /SPI0_CS_DDS -> /Relais1
- U101 pad 27: /SPI0_CS_CAN1 -> /Relais2
- U101 pad 29: /CD_SD -> /SPI0_CS_DDS
- U101 pad 4: /SPI0_CS_CAN2 -> unconnected-(U101-Pad4)
- U101 pad 9: /R1 -> unconnected-(U101-Pad9)
- U1301 pad 3: Net-(C45-Pad1) -> Net-(C1301-Pad1)
- U1301 pad 6: Net-(J23-Pad2) -> /CAN1/CANL
- U1301 pad 7: Net-(J23-Pad1) -> /CAN1/CANH
- U1302 pad 7: Net-(C46-Pad1) -> Net-(C1302-Pad1)
- U1302 pad 8: Net-(C47-Pad1) -> Net-(C1303-Pad1)
- U1401 pad 1: Net-(C50-Pad2) -> Net-(C1402-Pad2)
- U1401 pad 3: Net-(C49-Pad1) -> Net-(C1401-Pad1)
- U1701 pad 10: Net-(J26-Pad4) -> Net-(J1701-Pad1)
- U1701 pad 11: Net-(J26-Pad3) -> Net-(J1701-Pad2)
- U1701 pad 12: Net-(J26-Pad2) -> Net-(J1701-Pad3)
- U1701 pad 13: Net-(J26-Pad1) -> Net-(J1701-Pad4)
- U1701 pad 14: Net-(C56-Pad1) -> Net-(C1701-Pad1)
- U1701 pad 2: /DOUT1_LS -> /DOUT4_LS
- U1701 pad 3: /DOUT2_LS -> /DOUT3_LS
- U1701 pad 4: /DOUT3_LS -> /DOUT2_LS
- U1701 pad 5: /DOUT4_LS -> /DOUT1_LS
- U1901 pad 1: Net-(C59-Pad1) -> Net-(C1901-Pad1)
- U1901 pad 2: Net-(C59-Pad2) -> Net-(C1901-Pad2)
- U201 pad 5: Net-(R4-Pad2) -> /Battery/SCL_
- U201 pad 6: Net-(R3-Pad2) -> /Battery/SDA_
- U201 pad 7: Net-(R4-Pad2) -> /Battery/SDA_
- U201 pad 8: Net-(R4-Pad2) -> /Battery/SDA_
- U202 pad 6: Net-(R4-Pad2) -> /Battery/SCL_
- U202 pad 7: Net-(R3-Pad2) -> /Battery/SDA_
- U203 pad 1: Net-(U4-Pad1) -> Net-(U203-Pad1)
- U203 pad 4: Net-(R3-Pad2) -> /Battery/SDA_
- U203 pad 5: Net-(R4-Pad2) -> /Battery/SCL_
- U204 pad 1: Net-(Q1-Pad1) -> unconnected-(U204-Pad1)
- U204 pad 2: /Battery/BAT+ -> unconnected-(U204-Pad2)
- U204 pad 3: Net-(U4-Pad1) -> unconnected-(U204-Pad3)
- U204 pad 5: unconnected-(U5-Pad5) -> Net-(U203-Pad1)
- U204 pad 6: unconnected-(U5-Pad6) -> /Battery/BAT+
- U204 pad 7: unconnected-(U5-Pad7) -> Net-(Q201-Pad1)
- U2201 pad 1: Net-(C65-Pad1) -> Net-(C2201-Pad1)
- U2201 pad 2: Net-(C65-Pad2) -> Net-(C2201-Pad2)
- U2302 pad 3: Net-(C69-Pad1) -> Net-(C2303-Pad1)
- U2302 pad 4: Net-(C68-Pad2) -> Net-(C2302-Pad2)
- U2302 pad 8: Net-(C67-Pad1) -> Net-(C2301-Pad1)
- U601 pad 6: Net-(J19-Pad2) -> /CAN2/CANL
- U601 pad 7: Net-(J19-Pad1) -> /CAN2/CANH
- U801 pad 13: Net-(J20-Pad2) -> /UART to RS232/RX1
- U801 pad 14: Net-(J20-Pad1) -> /UART to RS232/TX1
- U801 pad 7: Net-(J21-Pad1) -> /UART to RS232/TX2
- U801 pad 8: Net-(J21-Pad2) -> /UART to RS232/RX2
- Y1301 pad 1: Net-(C46-Pad1) -> Net-(C1302-Pad1)
- Y1301 pad 2: Net-(C47-Pad1) -> Net-(C1303-Pad1)
Routing:
- net /I2C0_SDA: track 0.00 -> 312.1 mm, vias 0 -> 10
- net /I2C0_SCL: track 0.00 -> 305.7 mm, vias 0 -> 6
- net +5V: track 0.00 -> 292.1 mm, vias 0 -> 3
- net +3V3: track 0.00 -> 222.6 mm, vias 0 -> 22
- net GND: track 0.00 -> 141.4 mm, vias 0 -> 96
- net /UART0_TX: track 0.00 -> 107.1 mm, vias 0 -> 2
- net /VDC_EN: track 0.00 -> 103.8 mm, vias 0 -> 1
- net VCC: track 0.00 -> 98.2 mm, vias 0 -> 3
- net /UART0_RX: track 0.00 -> 94.3 mm
- net VDC: track 0.00 -> 93.2 mm, vias 0 -> 2
- net /SPI0_MOSI: track 0.00 -> 83.4 mm, vias 0 -> 5
- net /SPI0_SCK: track 0.00 -> 81.9 mm, vias 0 -> 5
- net /Relais2: track 0.00 -> 77.4 mm, vias 0 -> 1
- net /VCC_EN: track 0.00 -> 69.5 mm, vias 0 -> 1
- net /SPI0_CS_DDS: track 0.00 -> 68.4 mm, vias 0 -> 1
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- added copper zone on F.Cu, net +3V3
- added copper zone on F.Cu, net +5V
- added copper zone on F.Cu, net +5VD
- added copper zone on F.Cu, net /Power1/SW
- added copper zone on F.Cu, net /Power2/SW
- added copper zone on B.Cu, net GND
- added copper zone on F.Cu, net GND
- added copper zone on B.Cu, net GNDD
Other:
- board outline added: 100 x 100 mm
- board text added: "Gister embeddedBridge V1.0"
