File: embeddedBridge.kicad_sch (KiCad schematic)
At the start: 26 parts, among them J1 AOUT, J10 IO2, J11 R1, J12 R2, J13 R3, J14 R4, J2 I2C1, J3 I2C0, J4 Debug, J5 PWR, J6 DOUT1, J7 FOUT, J8 IO1, J9 DOUT2, SW1 RESET, U1 Pico

Commit message: layout
Parts:
- removed D1: D_Schottky, Diode_SMD:D_SMA-SMB_Universal_Handsoldering, symbol Device:D_Schottky
- removed J10: IO2, Connector_PinHeader_2.54mm:PinHeader_1x03_P2.54mm_Vertical, symbol Connector:Conn_01x03_Female
- removed J11: R1, Connector_PinHeader_2.54mm:PinHeader_1x03_P2.54mm_Vertical, symbol Connector:Conn_01x03_Female
- removed J12: R2, Connector_PinHeader_2.54mm:PinHeader_1x03_P2.54mm_Vertical, symbol Connector:Conn_01x03_Female
- removed J13: R3, Connector_PinHeader_2.54mm:PinHeader_1x03_P2.54mm_Vertical, symbol Connector:Conn_01x03_Female
- removed J14: R4, Connector_PinHeader_2.54mm:PinHeader_1x03_P2.54mm_Vertical, symbol Connector:Conn_01x03_Female
- removed J5: PWR, Connector_PinHeader_2.54mm:PinHeader_1x05_P2.54mm_Vertical, symbol Connector:Conn_01x05_Female
- removed J8: IO1, Connector_PinHeader_2.54mm:PinHeader_1x03_P2.54mm_Vertical, symbol Connector:Conn_01x03_Female
- removed J9: DOUT2, Connector_PinHeader_2.54mm:PinHeader_1x05_P2.54mm_Vertical, symbol Connector:Conn_01x05_Female
- removed JP2: DOUT1, Jumper:SolderJumper-2_P1.3mm_Bridged_Pad1.0x1.5mm, symbol Jumper:SolderJumper_2_Bridged
- removed JP3: DOUT2, Jumper:SolderJumper-2_P1.3mm_Bridged_Pad1.0x1.5mm, symbol Jumper:SolderJumper_2_Bridged
- removed JP4: DOUT3, Jumper:SolderJumper-2_P1.3mm_Bridged_Pad1.0x1.5mm, symbol Jumper:SolderJumper_2_Bridged
- removed JP5: DOUT4, Jumper:SolderJumper-2_P1.3mm_Bridged_Pad1.0x1.5mm, symbol Jumper:SolderJumper_2_Bridged
- added D101: 1N5819, Diode_SMD:D_SOD-323, symbol Diode:1N5819
- added H101, H102, H103, H104: MountingHole_Pad, MountingHole:MountingHole_3.2mm_M3_DIN965_Pad, symbol Mechanical:MountingHole_Pad
- added J105: VCC, Connector_PinHeader_2.54mm:PinHeader_1x02_P2.54mm_Vertical, symbol Connector:Conn_01x02_Female
- added J108: CAN1, Connector_PinHeader_2.54mm:PinHeader_1x03_P2.54mm_Vertical, symbol Connector:Conn_01x03_Female
- added J109: CAN2, Connector_PinHeader_2.54mm:PinHeader_1x03_P2.54mm_Vertical, symbol Connector:Conn_01x03_Female
- added J110: VDC, Connector_PinHeader_2.54mm:PinHeader_1x02_P2.54mm_Vertical, symbol Connector:Conn_01x02_Female
- added J111: R1_1, Connector_PinHeader_2.54mm:PinHeader_1x03_P2.54mm_Vertical, symbol Connector:Conn_01x03_Female
- added J112: R1_2, Connector_PinHeader_2.54mm:PinHeader_1x03_P2.54mm_Vertical, symbol Connector:Conn_01x03_Female
- added J113: R2_1, Connector_PinHeader_2.54mm:PinHeader_1x03_P2.54mm_Vertical, symbol Connector:Conn_01x03_Female
- added J114: R2_2, Connector_PinHeader_2.54mm:PinHeader_1x03_P2.54mm_Vertical, symbol Connector:Conn_01x03_Female
- added J115: RS232_2, Connector_PinHeader_2.54mm:PinHeader_1x03_P2.54mm_Vertical, symbol Connector:Conn_01x03_Female
- added J116: RS232_1, Connector_PinHeader_2.54mm:PinHeader_1x03_P2.54mm_Vertical, symbol Connector:Conn_01x03_Female
- added J117: +3V3, Connector_PinHeader_2.54mm:PinHeader_1x02_P2.54mm_Vertical, symbol Connector:Conn_01x02_Female
- added J118: +5V, Connector_PinHeader_2.54mm:PinHeader_1x02_P2.54mm_Vertical, symbol Connector:Conn_01x02_Female
- J102: renamed from J2; footprint Connector_JST:JST_PH_B2B-PH-K_1x02_P2.00mm_Vertical -> Connector_JST:JST_PH_B3B-PH-K_1x03_P2.00mm_Vertical
- TP101: renamed from TP1; value TestPoint -> +3V3
- TP102: renamed from TP2; value TestPoint -> DDS
- renumbered J1 to J101, J3 to J103, J4 to J104, J6 to J106, J7 to J107, JP1 to JP101, R1 to R101, R2 to R102, SW1 to SW101, U1 to U101
Connections:
- net R2 is gone; now on net SPI0_CS_SD: U101.10 (GPIO7)
- net R3 is gone; now on net SPI0_CS_CAN2: U101.19 (GPIO14)
- net R4 is gone; now on net SPI0_CS_CAN1: U101.20 (GPIO15)
- net +3V3: now also J117.1 (Pin_1)
- net +5V: now also D101.2 (A), J118.1 (Pin_1)
- net CD_SD: now also U101.22 (GPIO17); no longer U101.29 (GPIO22)
- net GND: now also J105.2 (Pin_2), J108.3 (Pin_3), J109.3 (Pin_3), J110.2 (Pin_2), J115.3 (Pin_3), J116.3 (Pin_3), J117.2 (Pin_2), J118.2 (Pin_2)
- net Relais1/COM1: now also J111.2 (Pin_2)
- net Relais1/COM2: now also J112.2 (Pin_2)
- net Relais1/NC1: now also J111.3 (Pin_3)
- net Relais1/NC2: now also J112.3 (Pin_3)
- net Relais1/NO1: now also J111.1 (Pin_1)
- net Relais1/NO2: now also J112.1 (Pin_1)
- net SPI0_CS_CAN1: no longer U101.27 (GPIO21)
- net SPI0_CS_CAN2: no longer U101.4 (GPIO2)
- net SPI0_CS_DDS: now also U101.29 (GPIO22); no longer U101.26 (GPIO20)
- net SPI0_CS_SD: no longer U101.22 (GPIO17)
- net VCC: now also J105.1 (Pin_1)
- net VDC: now also J110.1 (Pin_1)
- net VSYS: now also D101.1 (K)
- net R1: no longer names the net of U101.9 (GPIO6)
- new net CAN1/CANH: J108.1 (Pin_1)
- new net CAN1/CANL: J108.2 (Pin_2)
- new net CAN2/CANH: J109.1 (Pin_1)
- new net CAN2/CANL: J109.2 (Pin_2)
- new net Relais1: U101.26 (GPIO20)
- new net Relais2: U101.27 (GPIO21)
- new net Relais2/COM1: J113.2 (Pin_2)
- new net Relais2/COM2: J114.2 (Pin_2)
- new net Relais2/NC1: J113.3 (Pin_3)
- new net Relais2/NC2: J114.3 (Pin_3)
- new net Relais2/NO1: J113.1 (Pin_1)
- new net Relais2/NO2: J114.1 (Pin_1)
- new net UART to RS232/RX1: J116.2 (Pin_2)
- new net UART to RS232/RX2: J115.2 (Pin_2)
- new net UART to RS232/TX1: J116.1 (Pin_1)
- new net UART to RS232/TX2: J115.1 (Pin_1)
- no-connect marks 13 -> 25
Other:
- sheet Power renamed Power1
- sheet Relais renamed Relais1
- added sheet Power2 (Power.kicad_sch)
- added sheet Relais2 (Relais.kicad_sch)
- added sheet USB (USB.kicad_sch)
- sheet ADC1 ports: added none; removed AOUT1, AOUT2, AOUT3
- sheet CAN1 ports: added CANH, CANL; removed none
- sheet CAN2 ports: added CANH, CANL; removed none
- sheet Power1 ports: added EN, OUT; removed EN1, EN2, OUT1, OUT2
- sheet Relais1 ports: added IN; removed COM3, COM4, IN1, IN2, IN3, IN4, NC3, NC4, NO3, NO4
- sheet UART to RS232 ports: added RX1, RX2, TX1, TX2; removed none
- note removed: "--- ToDo --- AOUT/DDS filter / ferit?"
- moved on the sheet: J106, J107, TP102
