File: Hardware/DDS.kicad_sch (KiCad schematic)
At the start: 6 parts, among them U1401 AD9833xRM, X1401 XO32

Commit message: add software
Parts:
- C1403: value 20p -> 22p
Changed lines of the file:
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@@
       (effects (font (size 1.27 1.27)) (justify left))
     )
-    (property "Value" "20p" (id 1) (at 170.18 114.2999 0)
+    (property "Value" "22p" (id 1) (at 170.18 114.2999 0)
       (effects (font (size 1.27 1.27)) (justify left))
     )
