File: Hardware/embeddedBridge.kicad_sch (KiCad schematic)
At the start: 30 parts, among them J101 AOUT, J102 I2C1, J103 I2C0, J104 Debug, J105 VCC, J106 DOUT1, J107 FOUT, J108 CAN1, J109 CAN2, J110 VDC, J111 R1_1, J112 R1_2, J113 R2_1, J114 R2_2, J115 RS232_2, J116 RS232_1, J117 +3V3, J118 +5V, SW101 RESET, U101 Pico

Commit message: add software
Other:
- moved on the sheet: D101, H101, H102, H103, H104, J101, J102, J103, J104, J105, J106, J107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
